File: KiCAD_project_folder/Synaps_PCB_2021/Power_Supply.kicad_sch (KiCad schematic)
At the start: 30 parts, among them J1 USB_C_Receptacle, Q2 Q_PMOS_DGS, U1 MAX14748BEWW+

Commit message: Added footprints to powersupply schematic and started placing components on PCB
Parts:
- BT2: footprint (none) -> Battery:BatteryHolder_Keystone_2462_2xAA
- C37, C38, C39, C40, C41, C42, C43, C44, C45, C46, C47: footprint (none) -> Capacitor_SMD:C_1206_3216Metric_Pad1.33x1.80mm_HandSolder
- D2: footprint (none) -> LED_SMD:LED_1206_3216Metric_Pad1.42x1.75mm_HandSolder
- J1: footprint Connector_USB:USB_C_Receptacle_HRO_TYPE-C-31-M-12 -> Connector_USB:USB_C_Receptacle_Amphenol_12401548E4-2A
- L4: footprint (none) -> Inductor_SMD:L_1206_3216Metric_Pad1.22x1.90mm_HandSolder
- R10, R11, R12, R2, R3, R4, R5, R9: footprint (none) -> Resistor_SMD:R_1206_3216Metric_Pad1.30x1.75mm_HandSolder
- U1: footprint 21-100122_W542C3+1_MXM -> MAX14748:MAX14748BEWW&plus_
Changed lines of the file:
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@@
     (property "Reference" "J1" (id 0) (at 37.0078 22.4282 0))
     (property "Value" "USB_C_Receptacle" (id 1) (at 37.0078 24.7396 0))
-    (property "Footprint" "Connector_USB:USB_C_Receptacle_HRO_TYPE-C-31-M-12" (id 2) (at 38.1 54.61 0)
+    (property "Footprint" "Connector_USB:USB_C_Receptacle_Amphenol_12401548E4-2A" (id 2) (at 38.1 54.61 0)
       (effects (font (size 1.27 1.27)) hide)
     )
@@
     (property "Reference" "R10" (id 0) (at 160.02 89.535 90))
     (property "Value" "4.7K" (id 1) (at 160.655 87.63 90))
-    (property "Footprint" "" (id 2) (at 160.401 92.456 90)
+    (property "Footprint" "Resistor_SMD:R_1206_3216Metric_Pad1.30x1.75mm_HandSolder" (id 2) (at 160.401 92.456 90)
       (effects (font (size 1.27 1.27)) hide)
     )
@@
     (property "Reference" "C45" (id 0) (at 220.98 82.55 90))
     (property "Value" "1uF" (id 1) (at 220.98 85.09 90))
-    (property "Footprint" "" (id 2) (at 224.79 79.7052 0)
+    (property "Footprint" "Capacitor_SMD:C_1206_3216Metric_Pad1.33x1.80mm_HandSolder" (id 2) (at 224.79 79.7052 0)
       (effects (font (size 1.27 1.27)) hide)
     )
@@
     (property "Reference" "C44" (id 0) (at 161.29 71.755 90))
     (property "Value" "1uF" (id 1) (at 161.29 80.01 90))
-    (property "Footprint" "" (id 2) (at 165.1 77.1652 0)
+    (property "Footprint" "Capacitor_SMD:C_1206_3216Metric_Pad1.33x1.80mm_HandSolder" (id 2) (at 165.1 77.1652 0)
       (effects (font (size 1.27 1.27)) hide)
     )
@@
     (property "Reference" "R12" (id 0) (at 217.805 99.695 90))
     (property "Value" "4.7K" (id 1) (at 217.805 101.6 90))
-    (property "Footprint" "" (id 2) (at 218.059 103.124 90)
+    (property "Footprint" "Resistor_SMD:R_1206_3216Metric_Pad1.30x1.75mm_HandSolder" (id 2) (at 218.059 103.124 90)
       (effects (font (size 1.27 1.27)) hide)
     )
@@
       (effects (font (size 1.27 1.27)) (justify left))
     )
-    (property "Footprint" "" (id 2) (at 110.49 68.961 90)
+    (property "Footprint" "Battery:BatteryHolder_Keystone_2462_2xAA" (id 2) (at 110.49 68.961 90)
       (effects (font (size 1.27 1.27)) hide)
     )
@@
     (property "Reference" "C42" (id 0) (at 160.655 102.87 90))
     (property "Value" "0.1uF" (id 1) (at 160.655 104.775 90))
-    (property "Footprint" "" (id 2) (at 164.465 100.0252 0)
+    (property "Footprint" "Capacitor_SMD:C_1206_3216Metric_Pad1.33x1.80mm_HandSolder" (id 2) (at 164.465 100.0252 0)
       (effects (font (size 1.27 1.27)) hide)
     )
@@
       (effects (font (size 1.524 1.524)))
     )
-    (property "Footprint" "21-100122_W542C3+1_MXM" (id 2) (at 187.96 37.084 0)
+    (property "Footprint" "MAX14748:MAX14748BEWW&plus_" (id 2) (at 187.96 37.084 0)
       (effects (font (size 1.524 1.524)) hide)
     )
@@
     (property "Reference" "D2" (id 0) (at 226.695 85.725 0))
     (property "Value" "LED" (id 1) (at 226.695 91.44 0))
-    (property "Footprint" "" (id 2) (at 226.06 88.265 0)
+    (property "Footprint" "LED_SMD:LED_1206_3216Metric_Pad1.42x1.75mm_HandSolder" (id 2) (at 226.06 88.265 0)
       (effects (font (size 1.27 1.27)) hide)
     )
@@
     (property "Reference" "C46" (id 0) (at 238.76 73.66 90))
     (property "Value" "0.1uF" (id 1) (at 247.015 73.66 90))
-    (property "Footprint" "" (id 2) (at 244.1702 77.47 0)
+    (property "Footprint" "Capacitor_SMD:C_1206_3216Metric_Pad1.33x1.80mm_HandSolder" (id 2) (at 244.1702 77.47 0)
       (effects (font (size 1.27 1.27)) hide)
     )
@@
     (property "Reference" "C40" (id 0) (at 145.415 87.63 90))
     (property "Value" "1uF" (id 1) (at 145.415 90.17 90))
-    (property "Footprint" "" (id 2) (at 149.225 94.9452 0)
+    (property "Footprint" "Capacitor_SMD:C_1206_3216Metric_Pad1.33x1.80mm_HandSolder" (id 2) (at 149.225 94.9452 0)
       (effects (font (size 1.27 1.27)) hide)
     )
@@
     (property "Reference" "C47" (id 0) (at 251.46 73.66 90))
     (property "Value" "10uF" (id 1) (at 260.985 73.66 90))
-    (property "Footprint" "" (id 2) (at 256.8702 77.47 0)
+    (property "Footprint" "Capacitor_SMD:C_1206_3216Metric_Pad1.33x1.80mm_HandSolder" (id 2) (at 256.8702 77.47 0)
       (effects (font (size 1.27 1.27)) hide)
     )
@@
     (property "Reference" "R3" (id 0) (at 154.305 44.45 90))
     (property "Value" "4.7K" (id 1) (at 156.21 44.45 90))
-    (property "Footprint" "" (id 2) (at 157.734 44.196 90)
+    (property "Footprint" "Resistor_SMD:R_1206_3216Metric_Pad1.30x1.75mm_HandSolder" (id 2) (at 157.734 44.196 90)
       (effects (font (size 1.27 1.27)) hide)
     )
@@
     (property "Reference" "C39" (id 0) (at 128.27 65.405 90))
     (property "Value" "10uF" (id 1) (at 130.81 66.04 90))
-    (property "Footprint" "" (id 2) (at 134.9248 69.85 0)
+    (property "Footprint" "Capacitor_SMD:C_1206_3216Metric_Pad1.33x1.80mm_HandSolder" (id 2) (at 134.9248 69.85 0)
       (effects (font (size 1.27 1.27)) hide)
     )
@@
     (property "Reference" "R5" (id 0) (at 218.44 108.585 90))
     (property "Value" "4.7K" (id 1) (at 218.44 110.49 90))
-    (property "Footprint" "" (id 2) (at 218.694 105.664 90)
+    (property "Footprint" "Resistor_SMD:R_1206_3216Metric_Pad1.30x1.75mm_HandSolder" (id 2) (at 218.694 105.664 90)
       (effects (font (size 1.27 1.27)) hide)
     )
@@
     (property "Reference" "C37" (id 0) (at 127 86.36 90))
     (property "Value" "22uF" (id 1) (at 117.475 86.36 90))
-    (property "Footprint" "" (id 2) (at 121.5898 90.17 0)
+    (property "Footprint" "Capacitor_SMD:C_1206_3216Metric_Pad1.33x1.80mm_HandSolder" (id 2) (at 121.5898 90.17 0)
       (effects (font (size 1.27 1.27)) hide)
     )
@@
     (property "Reference" "C41" (id 0) (at 153.035 66.04 90))
     (property "Value" "0.1uF" (id 1) (at 154.94 66.04 90))
-    (property "Footprint" "" (id 2) (at 147.6248 69.85 0)
+    (property "Footprint" "Capacitor_SMD:C_1206_3216Metric_Pad1.33x1.80mm_HandSolder" (id 2) (at 147.6248 69.85 0)
       (effects (font (size 1.27 1.27)) hide)
     )
@@
     (property "Reference" "R2" (id 0) (at 142.24 49.53 90))
     (property "Value" "10K" (id 1) (at 142.24 52.07 90))
-    (property "Footprint" "" (id 2) (at 142.494 54.864 90)
+    (property "Footprint" "Resistor_SMD:R_1206_3216Metric_Pad1.30x1.75mm_HandSolder" (id 2) (at 142.494 54.864 90)
       (effects (font (size 1.27 1.27)) hide)
     )
@@
     (property "Reference" "C43" (id 0) (at 155.575 48.26 90))
     (property "Value" "3.9nF" (id 1) (at 155.575 50.165 90))
-    (property "Footprint" "" (id 2) (at 159.385 54.3052 0)
+    (property "Footprint" "Capacitor_SMD:C_1206_3216Metric_Pad1.33x1.80mm_HandSolder" (id 2) (at 159.385 54.3052 0)
       (effects (font (size 1.27 1.27)) hide)
     )
@@
     (property "Reference" "R4" (id 0) (at 214.63 71.755 90))
     (property "Value" "4.7K" (id 1) (at 214.63 73.66 90))
-    (property "Footprint" "" (id 2) (at 214.884 75.184 90)
+    (property "Footprint" "Resistor_SMD:R_1206_3216Metric_Pad1.30x1.75mm_HandSolder" (id 2) (at 214.884 75.184 90)
       (effects (font (size 1.27 1.27)) hide)
     )
@@
     (property "Reference" "R11" (id 0) (at 165.735 38.1 90))
     (property "Value" "10K" (id 1) (at 161.29 38.1 90))
-    (property "Footprint" "" (id 2) (at 162.179 37.846 90)
+    (property "Footprint" "Resistor_SMD:R_1206_3216Metric_Pad1.30x1.75mm_HandSolder" (id 2) (at 162.179 37.846 90)
       (effects (font (size 1.27 1.27)) hide)
     )
@@
     (property "Reference" "L4" (id 0) (at 262.255 64.135 0))
     (property "Value" "INDUCTOR" (id 1) (at 262.255 66.04 0))
-    (property "Footprint" "" (id 2) (at 262.255 68.58 0)
+    (property "Footprint" "Inductor_SMD:L_1206_3216Metric_Pad1.22x1.90mm_HandSolder" (id 2) (at 262.255 68.58 0)
       (effects (font (size 1.27 1.27)) hide)
     )
@@
     (property "Reference" "R9" (id 0) (at 218.44 92.71 90))
     (property "Value" "1K" (id 1) (at 218.44 90.805 90))
-    (property "Footprint" "" (id 2) (at 219.329 87.249 90)
+    (property "Footprint" "Resistor_SMD:R_1206_3216Metric_Pad1.30x1.75mm_HandSolder" (id 2) (at 219.329 87.249 90)
       (effects (font (size 1.27 1.27)) hide)
     )
@@
     (property "Reference" "C38" (id 0) (at 139.7 85.725 90))
     (property "Value" "0.1uF" (id 1) (at 130.175 85.725 90))
-    (property "Footprint" "" (id 2) (at 134.2898 89.535 0)
-      (effects (font (size 1.27 1.27)) hide)
-    )
+    (property "Footprint" "Capacitor_SMD:C_1206_3216Metric_Pad1.33x1.80mm_HandSolder" (id 2) (at 134.2898 89.535 0)
+      (effects (font (size 1.27 1.27)) hide)
+    )
