File: KiCAD_project_folder/Synaps_PCB_2021/Power_Supply.kicad_sch (KiCad schematic)
At the start: 23 parts, among them J1 USB_C_Receptacle, U4 1101M2S3CQE2, U5 1101M2S3CQE2

Commit message: wip
Other:
- note added: "I2C interface for battery charger"
Changed lines of the file:
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@@
+    (stroke (width 0) (type default) (color 0 0 0 0))
+  )
+  (polyline (pts (xy 246.38 16.51) (xy 246.38 41.91))
     (stroke (width 0) (type default) (color 0 0 0 0))
   )
@@
     (stroke (width 0) (type default) (color 0 0 0 0))
   )
+  (wire (pts (xy 257.81 27.94) (xy 267.97 27.94))
+    (stroke (width 0) (type default) (color 0 0 0 0))
+  )
   (wire (pts (xy 76.2 97.79) (xy 80.01 97.79))
+    (stroke (width 0) (type default) (color 0 0 0 0))
+  )
+  (polyline (pts (xy 279.4 41.91) (xy 246.38 41.91))
     (stroke (width 0) (type default) (color 0 0 0 0))
   )
@@
     (stroke (width 0.508) (type default) (color 0 0 0 0))
   )
+  (wire (pts (xy 257.81 20.32) (xy 275.59 20.32))
+    (stroke (width 0) (type default) (color 0 0 0 0))
+  )
   (wire (pts (xy 115.57 27.94) (xy 128.27 27.94))
     (stroke (width 0) (type default) (color 0 0 0 0))
@@
     (stroke (width 0) (type default) (color 0 0 0 0))
   )
+  (wire (pts (xy 257.81 31.75) (xy 267.97 31.75))
+    (stroke (width 0) (type default) (color 0 0 0 0))
+  )
   (wire (pts (xy 64.77 29.21) (xy 85.09 29.21))
     (stroke (width 0) (type default) (color 0 0 0 0))
@@
     (stroke (width 0) (type default) (color 0 0 0 0))
   )
+  (wire (pts (xy 257.81 39.37) (xy 267.97 39.37))
+    (stroke (width 0) (type default) (color 0 0 0 0))
+  )
   (wire (pts (xy 59.69 46.99) (xy 59.69 49.53))
     (stroke (width 0) (type default) (color 0 0 0 0))
@@
     (stroke (width 0) (type default) (color 0 0 0 0))
   )
+  (polyline (pts (xy 246.38 16.51) (xy 279.4 16.51))
+    (stroke (width 0) (type default) (color 0 0 0 0))
+  )
   (wire (pts (xy 21.59 138.43) (xy 35.56 138.43))
     (stroke (width 0) (type default) (color 0 0 0 0))
@@
     (stroke (width 0) (type default) (color 0 0 0 0))
   )
+  (wire (pts (xy 257.81 35.56) (xy 267.97 35.56))
+    (stroke (width 0) (type default) (color 0 0 0 0))
+  )
   (polyline (pts (xy 16.51 151.13) (xy 16.51 193.04))
     (stroke (width 0) (type default) (color 0 0 0 0))
@@
     (stroke (width 0) (type default) (color 0 0 0 0))
   )
+  (polyline (pts (xy 279.4 16.51) (xy 279.4 41.91))
+    (stroke (width 0) (type default) (color 0 0 0 0))
+  )
   (wire (pts (xy 222.25 96.52) (xy 231.14 96.52))
     (stroke (width 0) (type default) (color 0 0 0 0))
@@
   )
   (polyline (pts (xy 50.8 125.73) (xy 50.8 146.05))
+    (stroke (width 0) (type default) (color 0 0 0 0))
+  )
+  (wire (pts (xy 257.81 24.13) (xy 275.59 24.13))
     (stroke (width 0) (type default) (color 0 0 0 0))
   )
@@
     (effects (font (size 1.27 1.27)) (justify left bottom))
   )
+  (text "I2C interface for battery charger\n" (at 246.38 15.24 0)
+    (effects (font (size 1.27 1.27)) (justify left bottom))
+  )
   (text "USB OTG INTERFACE \n(NO INTERM. IC NEEDED)" (at 45.72 125.73 180)
     (effects (font (size 1.27 1.27)) (justify right bottom))
@@
     (effects (font (size 1.27 1.27)) (justify left bottom))
   )
+  (label "*INT" (at 264.16 27.94 0)
+    (effects (font (size 1.27 1.27)) (justify left bottom))
+  )
   (label "3V3_OUTREG" (at 213.36 139.7 0)
     (effects (font (size 1.27 1.27)) (justify left bottom))
@@
     (effects (font (size 1.27 1.27)) (justify left bottom))
   )
+  (label "I2CEXT0_SDA_out" (at 259.08 20.32 0)
+    (effects (font (size 1.27 1.27)) (justify left bottom))
+  )
   (label "BATT_CHARG" (at 54.61 171.45 90)
     (effects (font (size 1.27 1.27)) (justify left bottom))
@@
     (effects (font (size 1.27 1.27)) (justify left bottom))
   )
+  (label "SYSOK" (at 261.62 31.75 0)
+    (effects (font (size 1.27 1.27)) (justify left bottom))
+  )
   (label "TX1-" (at 54.61 62.23 0)
     (effects (font (size 1.27 1.27)) (justify left bottom))
@@
   )
   (label "5V_OUTREG" (at 209.55 58.42 0)
+    (effects (font (size 1.27 1.27)) (justify left bottom))
+  )
+  (label "LED_PMIC" (at 259.08 39.37 0)
     (effects (font (size 1.27 1.27)) (justify left bottom))
   )
@@
     (effects (font (size 1.27 1.27)) (justify left bottom))
   )
+  (label "I2CEXT0_SCL_out" (at 259.08 24.13 0)
+    (effects (font (size 1.27 1.27)) (justify left bottom))
+  )
+  (label "FSUS" (at 262.89 35.56 0)
+    (effects (font (size 1.27 1.27)) (justify left bottom))
+  )
   (label "TX1+" (at 54.61 64.77 0)
     (effects (font (size 1.27 1.27)) (justify left bottom))
@@
   (label "CC1" (at 71.12 34.29 0)
     (effects (font (size 1.27 1.27)) (justify left bottom))
+  )
+  (hierarchical_label "SYSOK" (shape input) (at 257.81 31.75 180)
+    (effects (font (size 1.27 1.27)) (justify right))
+  )
+  (hierarchical_label "LED_PMIC" (shape input) (at 257.81 39.37 180)
+    (effects (font (size 1.27 1.27)) (justify right))
   )
   (hierarchical_label "USB_D-" (shape bidirectional) (at 35.56 133.35 0)
     (effects (font (size 1.27 1.27)) (justify left))
   )
+  (hierarchical_label "SCL" (shape input) (at 257.81 24.13 180)
+    (effects (font (size 1.27 1.27)) (justify right))
+  )
+  (hierarchical_label "SDA" (shape bidirectional) (at 257.81 20.32 180)
+    (effects (font (size 1.27 1.27)) (justify right))
+  )
   (hierarchical_label "USB_D+" (shape bidirectional) (at 35.56 138.43 0)
     (effects (font (size 1.27 1.27)) (justify left))
   )
+  (hierarchical_label "*INT" (shape input) (at 257.81 27.94 180)
+    (effects (font (size 1.27 1.27)) (justify right))
+  )
+  (hierarchical_label "FSUS" (shape input) (at 257.81 35.56 180)
+    (effects (font (size 1.27 1.27)) (justify right))
+  )
   (symbol (lib_id "Connector:USB_C_Receptacle") (at 34.29 54.61 0) (unit 1)
