File: KiCAD_project_folder/Synaps_PCB_2021/Synaps_PCB_2021.kicad_pcb (KiCad board)
At the start: 4 copper layers, 101.6 x 101.6 mm, 55 parts, among them J1 USB_C_Receptacle, U10 BMI160, U2 ESP32-WROOM-32, U3 LTC2452ITS8-TRMPBF, U4 BMI160, U5 LTC2452ITS8-TRMPBF, U6 BMI160, U7 LTC2452ITS8-TRMPBF, U8 BMI160, U9 LTC2452ITS8-TRMPBF

Commit message: Added footprints to powersupply schematic and started placing components on PCB
Parts:
- removed U2: ESP32-WROOM-32, RF_Module:ESP32-WROOM-32
- added AE2: PBC ANT, RF_Antenna:Texas_SWRA117D_2.4GHz_Left, F.Cu at (-180.3, 101.6)
- added BT2: Battery_Cell, Battery:BatteryHolder_Keystone_2462_2xAA, F.Cu at (-189.8, 43.2)
- added C37: 22uF, Capacitor_SMD:C_1206_3216Metric_Pad1.33x1.80mm_HandSolder, F.Cu at (-109.2, 124.5)
- added C38: 0.1uF, Capacitor_SMD:C_1206_3216Metric_Pad1.33x1.80mm_HandSolder, F.Cu at (-97.8, 126.4)
- added C39: 10uF, Capacitor_SMD:C_1206_3216Metric_Pad1.33x1.80mm_HandSolder, F.Cu at (-103.5, 149.2)
- added C40: 1uF, Capacitor_SMD:C_1206_3216Metric_Pad1.33x1.80mm_HandSolder, F.Cu at (85.7, 51.4)
- added C41: 0.1uF, Capacitor_SMD:C_1206_3216Metric_Pad1.33x1.80mm_HandSolder, F.Cu at (-106.7, 168.3)
- added C42: 0.1uF, Capacitor_SMD:C_1206_3216Metric_Pad1.33x1.80mm_HandSolder, F.Cu at (88.9, 46.3)
- added C43: 3.9nF, Capacitor_SMD:C_1206_3216Metric_Pad1.33x1.80mm_HandSolder, F.Cu at (94.6, 46.3)
- added C44: 1uF, Capacitor_SMD:C_1206_3216Metric_Pad1.33x1.80mm_HandSolder, F.Cu at (80.0, 53.9)
- added C45: 1uF, Capacitor_SMD:C_1206_3216Metric_Pad1.33x1.80mm_HandSolder, F.Cu at (78.1, 67.9)
- added C46: 0.1uF, Capacitor_SMD:C_1206_3216Metric_Pad1.33x1.80mm_HandSolder, F.Cu at (-103.5, 117.5)
- added C47: 10uF, Capacitor_SMD:C_1206_3216Metric_Pad1.33x1.80mm_HandSolder, F.Cu at (-114.9, 137.2)
- added C48: 10µF, Capacitor_SMD:C_1206_3216Metric_Pad1.33x1.80mm_HandSolder, F.Cu at (-119.2, 114.8)
- added C49: TBD, Capacitor_SMD:C_1206_3216Metric_Pad1.33x1.80mm_HandSolder, F.Cu at (-125.2, 118.1)
- added C50: 0.1µF, Capacitor_SMD:C_1206_3216Metric_Pad1.33x1.80mm_HandSolder, F.Cu at (-131.3, 121.5)
- added C51: 0.1µF, Capacitor_SMD:C_1206_3216Metric_Pad1.33x1.80mm_HandSolder, F.Cu at (-137.3, 121.7)
- added C52: TBD, Capacitor_SMD:C_1206_3216Metric_Pad1.33x1.80mm_HandSolder, F.Cu at (-131.2, 114.8)
- added C53: 0.1µF, Capacitor_SMD:C_1206_3216Metric_Pad1.33x1.80mm_HandSolder, F.Cu at (-143.3, 128.4)
- added C54: NC, Capacitor_SMD:C_1206_3216Metric_Pad1.33x1.80mm_HandSolder, F.Cu at (-143.3, 125.0)
- added C55: NC, Capacitor_SMD:C_1206_3216Metric_Pad1.33x1.80mm_HandSolder, F.Cu at (-137.3, 128.4)
- added C56: NC, Capacitor_SMD:C_1206_3216Metric_Pad1.33x1.80mm_HandSolder, F.Cu at (-143.3, 121.7)
- added C57: 0.1µF, Capacitor_SMD:C_1206_3216Metric_Pad1.33x1.80mm_HandSolder, F.Cu at (-137.3, 125.0)
- added C58: 22pF/6.3V(10%), Capacitor_SMD:C_1206_3216Metric_Pad1.33x1.80mm_HandSolder, F.Cu at (-131.3, 124.8)
- added C59: 22pF/6.3V(10%), Capacitor_SMD:C_1206_3216Metric_Pad1.33x1.80mm_HandSolder, F.Cu at (-125.3, 121.5)
- added C60: 1µf, Capacitor_SMD:C_1206_3216Metric_Pad1.33x1.80mm_HandSolder, F.Cu at (-131.2, 118.1)
- added C61: 3.3nF/6.3V(10%), Capacitor_SMD:C_1206_3216Metric_Pad1.33x1.80mm_HandSolder, F.Cu at (-125.7, 114.3)
- added C62: 100pF, Capacitor_SMD:C_1206_3216Metric_Pad1.33x1.80mm_HandSolder, F.Cu at (-137.2, 118.1)
- added C63: 10nF/6.3V(10%), Capacitor_SMD:C_1206_3216Metric_Pad1.33x1.80mm_HandSolder, F.Cu at (-137.2, 114.8)
- added D2: LED, LED_SMD:LED_1206_3216Metric_Pad1.42x1.75mm_HandSolder, F.Cu at (92.1, 75.5)
- added IC2: ESP32-S2, ESP32-S2:ESP32-S2, F.Cu at (-194.9, 154.9)
- added L2: TBD, Inductor_SMD:L_1206_3216Metric_Pad1.22x1.90mm_HandSolder, F.Cu at (-211.5, 153.0)
- added L3: 2.0nH, Inductor_SMD:L_1206_3216Metric_Pad1.22x1.90mm_HandSolder, F.Cu at (-208.9, 148.6)
- added L4: INDUCTOR, Inductor_SMD:L_1206_3216Metric_Pad1.22x1.90mm_HandSolder, F.Cu at (103.5, 64.1)
- added R10: 4.7K, Resistor_SMD:R_1206_3216Metric_Pad1.30x1.75mm_HandSolder, F.Cu at (75.6, 62.2)
- added R11: 10K, Resistor_SMD:R_1206_3216Metric_Pad1.30x1.75mm_HandSolder, F.Cu at (103.5, 57.7)
- added R12: 4.7K, Resistor_SMD:R_1206_3216Metric_Pad1.30x1.75mm_HandSolder, F.Cu at (95.9, 66.0)
- added R2: 10K, Resistor_SMD:R_1206_3216Metric_Pad1.30x1.75mm_HandSolder, F.Cu at (94.6, 51.4)
- added R3: 4.7K, Resistor_SMD:R_1206_3216Metric_Pad1.30x1.75mm_HandSolder, F.Cu at (75.6, 56.4)
- added R9: 1K, Resistor_SMD:R_1206_3216Metric_Pad1.30x1.75mm_HandSolder, F.Cu at (88.9, 66.0)
- added U1: MAX14748BEWW+, MAX14748:MAX14748BEWW&plus_, F.Cu at (88.3, 57.8)
- C1: value CAP -> 1uF
- C10: value 10uF -> NC
- C11: value 0.1uF -> 1µF
- C9: value TBD -> 1µF
- J1: footprint Connector_USB:USB_C_Receptacle_HRO_TYPE-C-31-M-12 -> Connector_USB:USB_C_Receptacle_Amphenol_12401548E4-2A
- R4: value TBD -> 4.7K
- R5: value 100 -> 4.7K
- R6: value 100 -> 0R
- R7: value 100 -> 499R
- R8: value 100 -> 20K(5%)
- moved J1 154.6 mm to (69.2, 44.5)
- moved R4 137.2 mm to (95.9, 71.0)
- moved R5 122.3 mm to (87.0, 71.0)
- moved R8 25.7 mm to (-52.1, 80.6)
- moved R6 11.8 mm to (-46.4, 76.2)
- moved C11 3.26 mm to (-40.6, 71.8)
- moved R7 2.49 mm to (-27.3, 66.7)
- moved C10 0.44 mm to (-41.3, 64.8)
- moved C9 0.41 mm to (-34.9, 65.4)
Connections:
- C10 pad 2: GNDREF -> Earth
- C11 pad 1: GNDREF -> /Microcontroler/VDD_SDIO
- C11 pad 2: /Microcontroler/VDD33 -> Earth
- C9 pad 1: Net-(C9-Pad1) -> /Microcontroler/VDD33
- C9 pad 2: GNDREF -> Earth
- R4 pad 1: /Microcontroler/VDD33 -> Net-(R4-Pad1)
- R4 pad 2: Net-(C9-Pad1) -> +1V1
- R5 pad 1: unconnected-(R5-Pad1) -> Net-(R5-Pad1)
- R5 pad 2: /Microcontroler/MTDI -> +1V1
- R6 pad 1: unconnected-(R6-Pad1) -> /Microcontroler/XIN
- R6 pad 2: /Microcontroler/MTCK -> Net-(IC2-Pad45)
- R7 pad 1: unconnected-(R7-Pad1) -> /Microcontroler/GPIO1
- R7 pad 2: /Microcontroler/MTMS -> Net-(IC2-Pad41)
- R8 pad 1: unconnected-(R8-Pad1) -> Net-(C61-Pad1)
- R8 pad 2: /Microcontroler/MTDO -> Net-(C61-Pad2)
Routing:
- net Net-(D2-Pad1): track 0.00 -> 9.51 mm
- net +1V1: track 0.00 -> 7.70 mm
- net Net-(C43-Pad2): track 0.00 -> 2.92 mm
- added copper zone on In2.Cu, net +3V3
- added copper zone on B.Cu, net GNDREF
- added copper zone on F.Cu, net GNDREF
- added copper zone on In1.Cu, net GNDREF

Commit message: PCB ucontroller
Parts:
- added R4: 4.7K, Resistor_SMD:R_1206_3216Metric_Pad1.30x1.75mm_HandSolder, F.Cu at (154.7, 112.8)
- moved IC2 349.2 mm to (148.3, 90.7)
- moved BT2 338.9 mm to (139.3, 124.0)
- moved L2 324.8 mm to (109.2, 101.6)
- moved L3 310.0 mm to (101.0, 140.0)
- moved C47 299.9 mm to (179.6, 80.5)
- moved C37 283.0 mm to (170.2, 79.2)
- moved AE2 282.3 mm to (101.9, 107.5), turned to 90 degrees
- moved C46 278.4 mm to (173.5, 89.9)
- moved C54 276.9 mm to (133.1, 109.0)
- moved C53 276.7 mm to (132.8, 145.3), turned to 180 degrees
- moved C62 271.5 mm to (133.6, 98.8)
- moved C57 270.6 mm to (132.8, 140.0)
- moved C51 270.4 mm to (132.8, 134.1)
- moved C56 269.1 mm to (125.7, 117.3)
- moved U3 265.2 mm to (185.7, 67.3)
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Connections:
- net Net-(BT2-Pad1) renamed /Power Supply/V_BAT
- net Net-(R9-Pad1) renamed /Power Supply/LED_PMIC
- C11 pad 1: /Microcontroler/VDD_SDIO -> unconnected-(C11-Pad1)
- C14 pad 1: +3V3 -> +1V1
- C15 pad 1: +3V3 -> +1V1
- C16 pad 1: +3V3 -> +1V1
- C17 pad 1: VDD -> +1V1
- C22 pad 1: +3V3 -> +1V1
- C23 pad 1: +3V3 -> +1V1
- C24 pad 1: +3V3 -> +1V1
- C25 pad 1: VDD -> +1V1
- C3 pad 1: +3V3 -> +1V1
- C30 pad 1: +3V3 -> +1V1
- C31 pad 1: +3V3 -> +1V1
- C32 pad 1: +3V3 -> +1V1
- C33 pad 1: VDD -> +1V1
- C37 pad 1: Net-(C37-Pad1) -> +1V1
- C38 pad 1: Net-(C37-Pad1) -> +1V1
- C4 pad 1: +3V3 -> +1V1
- C5 pad 1: +3V3 -> +1V1
- C6 pad 1: VDD -> +1V1
- IC2 pad 25: /Microcontroler/GPIO16 -> /Microcontroler/USB_D-
- IC2 pad 26: /Microcontroler/VDD_SDIO -> /Microcontroler/USB_D+
- J1 pad A4: /Power Supply/VBUS_C -> /Power Supply/CHGIN
- J1 pad A6: /Power Supply/CDP -> /Microcontroler/USB_D+
- J1 pad A7: /Power Supply/CDN -> /Microcontroler/USB_D-
- J1 pad A9: /Power Supply/VBUS_C -> /Power Supply/CHGIN
- J1 pad B4: /Power Supply/VBUS_C -> /Power Supply/CHGIN
- J1 pad B5: /Power Supply/CC2 -> /Power Supply/VCONN
- J1 pad B6: /Power Supply/CDP -> /Microcontroler/USB_D+
- J1 pad B7: /Power Supply/CDN -> /Microcontroler/USB_D-
- J1 pad B8: /Power Supply/VBUS_C -> /Power Supply/SBUS2
- J1 pad B9: /Power Supply/VBUS_C -> /Power Supply/CHGIN
- J1 pad S1: GNDREF -> Net-(J1-PadS1)
- R10 pad 1: Net-(R10-Pad1) -> +1V1
- R10 pad 2: +1V1 -> /Power Supply/SDA
- R12 pad 1: Net-(R12-Pad1) -> /Power Supply/SCL
- R5 pad 1: Net-(R5-Pad1) -> /Power Supply/*INT
- TP2 pad 1: /Power Supply/CC2 -> /Power Supply/VCONN
- TP3 pad 1: /Power Supply/CDN -> /Microcontroler/USB_D-
- TP4 pad 1: /Power Supply/CDP -> /Microcontroler/USB_D+
- U1 pad A3: Net-(R3-Pad1) -> /Power Supply/SYSOK
- U1 pad B3: unconnected-(U1-PadB3) -> GNDREF
- U1 pad B6: Net-(C37-Pad1) -> +1V1
- U1 pad B7: Net-(C37-Pad1) -> +1V1
- U1 pad B8: Net-(C37-Pad1) -> +1V1
- U1 pad B9: Net-(C37-Pad1) -> +1V1
- U1 pad C1: unconnected-(U1-PadC1) -> /Power Supply/VCONN
- U1 pad C2: Net-(R10-Pad1) -> /Power Supply/SCL
- U1 pad C4: unconnected-(U1-PadC4) -> GNDREF
- U1 pad D1: unconnected-(U1-PadD1) -> /Power Supply/CC1
- U1 pad D2: Net-(R5-Pad1) -> /Power Supply/SDA
- U1 pad D3: Net-(R12-Pad1) -> /Power Supply/*INT
- U1 pad E5: Net-(R4-Pad1) -> unconnected-(U1-PadE5)
- U10 pad 8: VDD -> +1V1
- U3 pad 3: +3V3 -> +1V1
- U3 pad 4: +3V3 -> +1V1
- U4 pad 8: VDD -> +1V1
- U5 pad 3: +3V3 -> +1V1
- U5 pad 4: +3V3 -> +1V1
- U6 pad 8: VDD -> +1V1
- U7 pad 3: +3V3 -> +1V1
- U7 pad 4: +3V3 -> +1V1
- U8 pad 8: VDD -> +1V1
- U9 pad 3: +3V3 -> +1V1
- U9 pad 4: +3V3 -> +1V1
Routing:
- net Net-(D2-Pad1): track 9.51 -> 0.00 mm
- net +1V1: track 7.70 -> 0.00 mm
- net Net-(C43-Pad2): track 2.92 -> 0.00 mm
- added copper zone on In2.Cu, net +1V1
- removed copper zone on In2.Cu, net +3V3

Commit message: Redid schematic, fixed wrong setup
Parts:
- removed C12, C15, C16, C18, C19, C20, C23, C24, C26, C27, C28, C31, C32, C34, C35, C36: 0.1uF, Capacitor_SMD:C_1206_3216Metric_Pad1.33x1.80mm_HandSolder
- removed C13, C17, C21, C25, C29, C33: 100nF, Capacitor_SMD:C_1206_3216Metric_Pad1.33x1.80mm_HandSolder
- removed C14, C22, C30: 10uF, Capacitor_SMD:C_1206_3216Metric_Pad1.33x1.80mm_HandSolder
- removed C51, C53, C57: 0.1µF, Capacitor_SMD:C_1206_3216Metric_Pad1.33x1.80mm_HandSolder
- removed C55, C56: NC, Capacitor_SMD:C_1206_3216Metric_Pad1.33x1.80mm_HandSolder
- removed C60: 1µf, Capacitor_SMD:C_1206_3216Metric_Pad1.33x1.80mm_HandSolder
- removed C61: 3.3nF/6.3V(10%), Capacitor_SMD:C_1206_3216Metric_Pad1.33x1.80mm_HandSolder
- removed C62: 100pF, Capacitor_SMD:C_1206_3216Metric_Pad1.33x1.80mm_HandSolder
- removed C63: 10nF/6.3V(10%), Capacitor_SMD:C_1206_3216Metric_Pad1.33x1.80mm_HandSolder
- removed U10, U4, U6, U8: BMI160, BMI160:BMI160
- removed U5, U7, U9: LTC2452ITS8-TRMPBF, LTC2456:LTC2452ITS8-TRMPBF
- added U2: CD74HC4067M, Package_SO:SOIC-24W_7.5x15.4mm_P1.27mm, F.Cu at (-36.2, 59.7)
- U3: value LTC2452ITS8-TRMPBF -> AT25DF041x-UxN-x; footprint LTC2456:LTC2452ITS8-TRMPBF -> Package_CSP:WLCSP-8_1.58x1.63x0.35mm_Layout3x5_P0.35x0.4mm_Ball0.25mm_Pad0.25mm_NSMD
Connections:
- net /Microcontroler/GPIO0 renamed /Microcontroler/DAC_1
- net /Microcontroler/GPIO10 renamed /Microcontroler/SPICS1
- net /Microcontroler/GPIO15 renamed /Microcontroler/XTAL_32K_P
- net /Microcontroler/GPIO18 renamed Net-(IC2-Pad35)
- net /Microcontroler/GPIO2 renamed /Microcontroler/XTAL_32K_N
- net /Microcontroler/GPIO22 renamed /Microcontroler/SPI3_MOSI
- net /Microcontroler/GPIO23 renamed Net-(IC2-Pad36)
- net /Microcontroler/GPIO25 renamed /Connectors/CAN_BUS_OFF_ON
- net /Microcontroler/GPIO26 renamed /Connectors/CAN_BUS_CLK
- net /Microcontroler/GPIO32 renamed /Connectors/CAN_BUS_RX
- net /Microcontroler/GPIO33 renamed /Connectors/CAN_BUS_TX
- net /Microcontroler/GPIO4 renamed /Microcontroler/DAC_2
- net /Microcontroler/GPIO5 renamed Net-(IC2-Pad34)
- net /Microcontroler/GPIO6 renamed Net-(IC2-Pad31)
- net /Microcontroler/GPIO7 renamed Net-(IC2-Pad32)
- net Net-(C52-Pad1) renamed /Microcontroler/LNA_IN
- net Net-(C54-Pad1) renamed /Microcontroler/VDD3P3
- AE2 pad 1: Earth -> GNDREF
- C48 pad 1: /Microcontroler/VDD33 -> +1V1
- C48 pad 2: Earth -> unconnected-(C48-Pad2)
- C49 pad 2: Earth -> GNDREF
- C50 pad 1: /Microcontroler/VDD33 -> +1V1
- C50 pad 2: Earth -> unconnected-(C50-Pad2)
- C52 pad 2: Earth -> GNDREF
- C54 pad 2: Earth -> GNDREF
- C58 pad 2: Earth -> GNDREF
- C59 pad 2: Earth -> GNDREF
- C9 pad 1: /Microcontroler/VDD33 -> +1V1
- C9 pad 2: Earth -> unconnected-(C9-Pad2)
- D2 pad 2: unconnected-(D2-Pad2) -> /Microcontroler/LED_PMIC
- IC2 pad 1: /Microcontroler/VDD33 -> +1V1
- IC2 pad 10: /Microcontroler/GPIO34 -> /Microcontroler/I2CEXT0_SCL_out
- IC2 pad 11: /Microcontroler/GPIO35 -> /Microcontroler/LED_PMIC
- IC2 pad 16: /Microcontroler/GPIO27 -> /Microcontroler/GPIO11
- IC2 pad 17: /Microcontroler/GPIO14 -> /Microcontroler/FSUS
- IC2 pad 18: /Microcontroler/GPIO12 -> /Microcontroler/ADC2_CH1
- IC2 pad 19: /Microcontroler/VDD33 -> /Microcontroler/ADC2_CH1
- IC2 pad 20: /Microcontroler/GPIO13 -> +1V1
- IC2 pad 27: /Microcontroler/GPIO17 -> +1V1
- IC2 pad 28: /Microcontroler/GPIO9 -> /Microcontroler/GPIO21
- IC2 pad 30: /Microcontroler/GPIO11 -> /Microcontroler/VDD_SPI
- IC2 pad 33: /Microcontroler/GPIO8 -> /Microcontroler/SPICS0
- IC2 pad 37: /Microcontroler/VDD33 -> /Microcontroler/SPI3_CS1
- IC2 pad 38: /Microcontroler/GPIO19 -> /Microcontroler/SPI3_MISO
- IC2 pad 40: /Microcontroler/GPIO3 -> /Microcontroler/SPI3_CS0
- IC2 pad 41: Net-(IC2-Pad41) -> /Microcontroler/SPI3_CLK
- IC2 pad 42: /Microcontroler/GPIO21 -> /Microcontroler/SPI3_CS2
- IC2 pad 43: /Microcontroler/VDD33 -> /Connectors/JTAG_MTCK
- IC2 pad 44: /Microcontroler/XOUT -> /Connectors/JTAG_MTDO
- IC2 pad 45: Net-(IC2-Pad45) -> +1V1
- IC2 pad 46: /Microcontroler/VDD33 -> /Connectors/JTAG_MTMS
- IC2 pad 47: Net-(C61-Pad2) -> /Connectors/JTAG_MTDI
- IC2 pad 48: Net-(C61-Pad1) -> Net-(IC2-Pad48)
- IC2 pad 49: Earth -> /Connectors/U0RXD
- IC2 pad 5: /Microcontroler/SENSOR_VP -> /Microcontroler/ADC1_CH0
- IC2 pad 50: unconnected-(IC2-Pad50) -> /Microcontroler/SPI_CS3
- IC2 pad 51: unconnected-(IC2-Pad51) -> +1V1
- IC2 pad 52: unconnected-(IC2-Pad52) -> /Microcontroler/XOUT
- IC2 pad 53: unconnected-(IC2-Pad53) -> /Microcontroler/XTAL_P
- IC2 pad 54: unconnected-(IC2-Pad54) -> +1V1
- IC2 pad 55: unconnected-(IC2-Pad55) -> /Microcontroler/GPIO46
- IC2 pad 56: unconnected-(IC2-Pad56) -> /Microcontroler/CHIP_PU
- IC2 pad 57: unconnected-(IC2-Pad57) -> GNDREF
- IC2 pad 6: Net-(C55-Pad2) -> /Microcontroler/ADC1_CH1
- IC2 pad 7: Net-(C56-Pad1) -> /Microcontroler/*INT
- IC2 pad 8: /Microcontroler/SENSOR_VN -> /Microcontroler/*INT
- IC2 pad 9: /Microcontroler/CHIP_PU -> /Microcontroler/I2CEXT0_SCL_out
- L3 pad 1: /Microcontroler/VDD33 -> +1V1
- R10 pad 2: /Power Supply/SDA -> /Microcontroler/I2CEXT0_SCL_out
- R12 pad 1: /Power Supply/SCL -> /Microcontroler/I2CEXT0_SCL_out
- R4 pad 1: /Power Supply/SYSOK -> /Microcontroler/*INT
- R4 pad 1: Net-(R4-Pad1) -> /Microcontroler/*INT
- R5 pad 1: /Power Supply/*INT -> /Microcontroler/*INT
- R9 pad 1: /Power Supply/LED_PMIC -> /Microcontroler/LED_PMIC
- U1 pad A3: /Power Supply/SYSOK -> /Microcontroler/*INT
- U1 pad B2: unconnected-(U1-PadB2) -> /Microcontroler/FSUS
- U1 pad C2: /Power Supply/SCL -> /Microcontroler/I2CEXT0_SCL_out
- U1 pad D2: /Power Supply/SDA -> /Microcontroler/I2CEXT0_SCL_out
- U1 pad D3: /Power Supply/*INT -> /Microcontroler/*INT
- U1 pad D4: unconnected-(U1-PadD4) -> GNDREF
- U1 pad D5: unconnected-(U1-PadD5) -> GNDREF
- U1 pad D6: unconnected-(U1-PadD6) -> GNDREF
- U1 pad D7: unconnected-(U1-PadD7) -> GNDREF
- U1 pad D8: unconnected-(U1-PadD8) -> GNDREF
- U1 pad D9: unconnected-(U1-PadD9) -> GNDREF
- U1 pad E2: /Power Supply/LED_PMIC -> /Microcontroler/LED_PMIC
