File: KiCAD_project_folder/Synaps_PCB_2021/Synaps_PCB_2021.kicad_pcb (KiCad board)
At the start: 4 copper layers, 101.6 x 101.6 mm, 75 parts, among them IC2 ESP32-S2, J1 USB_C_Receptacle, J2 Conn_01x20_MountingPin, J3 Conn_01x20_MountingPin, Q2 Q_PMOS_DGS, SW2 SW_Push, SW3 SW_Push, SW4 SW_Push, U1 MAX14748BEWW+, U2 CD74HC4067M, U3 AT25DF041x-UxN-x, Y2 Crystal_GND24, Y3 32.768K

Commit message: Schematic update
Parts:
- added BT3: Battery_Cell, Battery:BatteryHolder_Keystone_2462_2xAA, F.Cu at (305.6, 94.2)
- added BT4: Battery_Cell, Battery:BatteryHolder_Keystone_2462_2xAA, F.Cu at (305.6, 23.3)
- added BT5: Battery_Cell, Battery:BatteryHolder_Keystone_2462_2xAA, F.Cu at (305.6, 57.8)
- added C12: 10uF, Capacitor_SMD:C_1206_3216Metric_Pad1.33x1.80mm_HandSolder, F.Cu at (305.2, 120.6)
- added C13: 0.1uF, Capacitor_SMD:C_1206_3216Metric_Pad1.33x1.80mm_HandSolder, F.Cu at (305.2, 124.0)
- added C14: 10uF, Capacitor_SMD:C_1206_3216Metric_Pad1.33x1.80mm_HandSolder, F.Cu at (305.2, 127.3)
- added C15: 0.1uF, Capacitor_SMD:C_1206_3216Metric_Pad1.33x1.80mm_HandSolder, F.Cu at (305.2, 130.7)
- added L4: L_Ferrite 60 Omh 1.5 A, Ferrite_THT:LairdTech_28C0236-0JW-10, F.Cu at (310.1, 123.4)
- C49: value TBD -> 19pF; footprint Capacitor_SMD:C_1206_3216Metric_Pad1.33x1.80mm_HandSolder -> Capacitor_SMD:C_01005_0402Metric
- C52: value TBD -> 16pF; footprint Capacitor_SMD:C_1206_3216Metric_Pad1.33x1.80mm_HandSolder -> Capacitor_SMD:C_01005_0402Metric_Pad0.57x0.30mm_HandSolder
- C7, C8: value 12.5pF -> 22pF
- J2: value Conn_01x20_MountingPin -> Conn_02x10_MountingPin; footprint Connector_PinHeader_2.00mm:PinHeader_1x20_P2.00mm_Vertical -> Connector_PinHeader_2.54mm:PinHeader_2x10_P2.54mm_Vertical_SMD
- L2: value TBD -> 0.5028nH
- L5: value L_Ferrite -> L_Ferrite 60 Omh 1.5 A
- Y2: value Crystal_GND24 -> 40 MHz
- Y3: value 32.768K -> 32.768 KHz
Connections:
- BT2 pad 1: /Power Supply/V_BAT -> Net-(BT2-+)
- C48 pad 2: unconnected-(C48-Pad2) -> GNDREF
- C50 pad 2: unconnected-(C50-Pad2) -> GNDREF
- C9 pad 2: unconnected-(C9-Pad2) -> GNDREF
- IC2 pad 10: /Microcontroler/I2CEXT0_SCL_out -> /Microcontroler/I2CEXT0_SDA_out
- IC2 pad 8: /Microcontroler/*INT -> /Microcontroler/SYSOK
- J1 pad B5: /Power Supply/VCONN -> /Power Supply/CC2
- TP2 pad 1: /Power Supply/VCONN -> /Power Supply/CC2
Routing:
- net /Power Supply/VCONN: track 119.6 -> 0.00 mm
- net /Power Supply/CC2: track 0.00 -> 119.6 mm
