File: KiCAD_project_folder/Synaps_PCB_2021/BQ24725RGRR.kicad_sch (KiCad schematic)
At the start: 1 part

Commit message: power supply structure rework
Parts:
- gave numbers to parts that had none: 1
Changed lines of the file:
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@@
 (kicad_sch (version 20211123) (generator eeschema)
   (paper "A4")
+  (title_block
+    (date "2022-11-14")
+  )
   (symbol (lib_id "BQ24725:BQ24725RGRR") (at 93.98 71.12 0) (unit 1)
     (in_bom yes) (on_board yes) (fields_autoplaced)
-    (property "Reference" "U?" (id 0) (at 127 61.8924 0)
+    (property "Reference" "U12" (id 0) (at 127 61.8924 0)
       (effects (font (size 1.524 1.524)))
     )
