File: KiCAD_project_folder/Synaps_PCB_2021/TPS25741ARSMR.kicad_sch (KiCad schematic)
At the start: 4 parts

Commit message: Added subcomponents for replacement charging circuit
Parts:
- U?: MPN (none) -> CDBA340L-HF; Supplier Link (none) -> https://www.digikey.ca/en/products/detail/comchip-technolog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
Changed lines of the file:
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@@
       (effects (font (size 1.524 1.524)) hide)
     )
-    (property "Datasheet" "" (id 3) (at 138.43 52.07 0)
-      (effects (font (size 1.524 1.524)))
+    (property "Datasheet" "https://www.comchiptech.com/admin/files/product/CDBA340L-HF%20RevC514368.pdf" (id 3) (at 138.43 52.07 0)
+      (effects (font (size 1.524 1.524)) hide)
+    )
+    (property "MPN" "CDBA340L-HF" (id 4) (at 138.43 52.07 0)
+      (effects (font (size 1.27 1.27)) hide)
+    )
+    (property "Supplier Link" "https://www.digikey.ca/en/products/detail/comchip-technology/CDBA340L-HF/3308142" (id 5) (at 138.43 52.07 0)
+      (effects (font (size 1.27 1.27)) hide)
     )
     (pin "1")

Commit message: power supply structure rework
Parts:
- gave numbers to parts that had none: 4
Changed lines of the file:
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@@
 (kicad_sch (version 20211123) (generator eeschema)
   (paper "A4")
+  (title_block
+    (date "2022-11-14")
+  )
   (symbol (lib_id "CDBA340L-HF:CDBA340L-HF") (at 138.43 52.07 0) (unit 1)
     (in_bom yes) (on_board yes) (fields_autoplaced)
-    (property "Reference" "U?" (id 0) (at 143.51 45.9793 0)
+    (property "Reference" "U6" (id 0) (at 143.51 45.9793 0)
       (effects (font (size 1.524 1.524)))
     )
@@
   (symbol (lib_id "CSD17310Q5A:CSD17310Q5A") (at 52.07 55.88 0) (unit 1)
     (in_bom yes) (on_board yes) (fields_autoplaced)
-    (property "Reference" "U?" (id 0) (at 74.93 46.6524 0)
+    (property "Reference" "U4" (id 0) (at 74.93 46.6524 0)
       (effects (font (size 1.524 1.524)))
     )
@@
   (symbol (lib_id "CSD17310Q5A:CSD17310Q5A") (at 203.2 58.42 0) (unit 1)
     (in_bom yes) (on_board yes) (fields_autoplaced)
-    (property "Reference" "U?" (id 0) (at 226.06 49.1924 0)
+    (property "Reference" "U7" (id 0) (at 226.06 49.1924 0)
       (effects (font (size 1.524 1.524)))
     )
@@
   (symbol (lib_id "TPS25741:TPS25741ARSMR") (at 114.3 87.63 0) (unit 1)
     (in_bom yes) (on_board yes) (fields_autoplaced)
-    (property "Reference" "U?" (id 0) (at 142.24 78.4024 0)
+    (property "Reference" "U5" (id 0) (at 142.24 78.4024 0)
       (effects (font (size 1.524 1.524)))
     )
