File: KiCAD_project_folder/Synaps_PCB_2021/TVS2201DRBR.kicad_sch (KiCad schematic)
At the start: 1 part

Commit message: power supply structure rework
Parts:
- gave numbers to parts that had none: 1
Changed lines of the file:
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@@
 (kicad_sch (version 20211123) (generator eeschema)
   (paper "A4")
+  (title_block
+    (date "2022-11-14")
+  )
   (symbol (lib_id "TVS2201:TVS2201DRBR") (at 111.76 88.9 0) (unit 1)
     (in_bom yes) (on_board yes) (fields_autoplaced)
-    (property "Reference" "U?" (id 0) (at 111.76 77.631 0))
+    (property "Reference" "U11" (id 0) (at 111.76 77.631 0))
     (property "Value" "TVS2201DRBR" (id 1) (at 111.76 80.1679 0))
     (property "Footprint" "TVS2201:IC_DRV8601DRBT" (id 2) (at 111.76 88.9 0)
