File: KiCAD_project_folder/Synaps_PCB_2021/Probes.kicad_sch (KiCad schematic)
At the start: 3 parts, among them J3 Conn_02x10_MountingPin, U2 CD74HC4067M, U9 74HCT4067PW_118

Commit message: power supply structure rework
Parts:
- removed U9: 74HCT4067PW_118, 74HCT4067PW-118:74HCT4067PW_118, symbol 74HCT4067PW-118:74HCT4067PW_118
Changed lines of the file:
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@@
   (title_block
     (title "Misca PCB")
-    (date "2022-06-17")
+    (date "2022-11-14")
     (rev "A2")
     (company "Club SynapsÉTS")
@@
     (pin "1")
   )
-  (symbol (lib_id "74HCT4067PW-118:74HCT4067PW_118") (at 99.06 121.92 0) (unit 1)
-    (in_bom yes) (on_board yes) (fields_autoplaced)
-    (property "Reference" "U9" (id 0) (at 119.38 112.6924 0)
-      (effects (font (size 1.524 1.524)))
-    )
-    (property "Value" "74HCT4067PW_118" (id 1) (at 119.38 115.6858 0)
-      (effects (font (size 1.524 1.524)))
-    )
-    (property "Footprint" "74HCT4067PW-118:74HCT4067PW_118" (id 2) (at 119.38 115.824 0)
-      (effects (font (size 1.524 1.524)) hide)
-    )
-    (property "Datasheet" "https://assets.nexperia.com/documents/data-sheet/74HC_HCT4067.pdf" (id 3) (at 99.06 121.92 0)
-      (effects (font (size 1.524 1.524)) hide)
-    )
-    (property "MPN" "74HCT4067PW,118" (id 4) (at 99.06 121.92 0)
-      (effects (font (size 1.27 1.27)) hide)
-    )
-    (property "Supplier Link" "https://www.digikey.ca/en/products/detail/nexperia-usa-inc/74HCT4067PW-118/1230918" (id 5) (at 99.06 121.92 0)
-      (effects (font (size 1.27 1.27)) hide)
-    )
-    (pin "1")
-    (pin "10")
-    (pin "11")
-    (pin "12")
-    (pin "13")
-    (pin "14")
-    (pin "15")
-    (pin "16")
-    (pin "17")
-    (pin "18")
-    (pin "19")
-    (pin "2")
-    (pin "20")
-    (pin "21")
-    (pin "22")
-    (pin "23")
-    (pin "24")
-    (pin "3")
-    (pin "4")
-    (pin "5")
-    (pin "6")
-    (pin "7")
-    (pin "8")
-    (pin "9")
-  )
   (symbol (lib_id "power:GNDREF") (at 142.24 90.17 0) (unit 1)

Commit message: wip
Parts:
- added U?: PI4IOE5V6416ZDEX, PI4IOE5V6416ZDEX_DIO, symbol PI4IOE5V6416ZDEX:PI4IOE5V6416ZDEX
- added U?: AD7490BCPZ, CP_32_2_ADI, symbol AD7490BCPZ:AD7490BCPZ
Changed lines of the file:
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@@
     (effects (font (size 1.27 1.27)) (justify right))
+  )
+  (symbol (lib_id "PI4IOE5V6416ZDEX:PI4IOE5V6416ZDEX") (at 38.1 124.46 0) (unit 1)
+    (in_bom yes) (on_board yes) (fields_autoplaced)
+    (property "Reference" "U?" (id 0) (at 66.04 113.03 0)
+      (effects (font (size 1.524 1.524)))
+    )
+    (property "Value" "PI4IOE5V6416ZDEX" (id 1) (at 66.04 116.84 0)
+      (effects (font (size 1.524 1.524)))
+    )
+    (property "Footprint" "PI4IOE5V6416ZDEX_DIO" (id 2) (at 38.1 124.46 0)
+      (effects (font (size 1.27 1.27) italic) hide)
+    )
+    (property "Datasheet" "PI4IOE5V6416ZDEX" (id 3) (at 38.1 124.46 0)
+      (effects (font (size 1.27 1.27) italic) hide)
+    )
+    (pin "1")
+    (pin "10")
+    (pin "11")
+    (pin "12")
+    (pin "13")
+    (pin "14")
+    (pin "15")
+    (pin "16")
+    (pin "17")
+    (pin "18")
+    (pin "19")
+    (pin "2")
+    (pin "20")
+    (pin "22")
+    (pin "24")
+    (pin "25")
+    (pin "3")
+    (pin "4")
+    (pin "5")
+    (pin "6")
+    (pin "7")
+    (pin "8")
+    (pin "9")
   )
   (symbol (lib_id "Connector_Generic_MountingPin:Conn_01x20_MountingPin") (at 219.71 60.96 0) (unit 1)
@@
     (pin "1")
   )
+  (symbol (lib_id "AD7490BCPZ:AD7490BCPZ") (at 129.54 111.76 0) (unit 1)
+    (in_bom yes) (on_board yes) (fields_autoplaced)
+    (property "Reference" "U?" (id 0) (at 162.56 100.33 0)
+      (effects (font (size 1.524 1.524)))
+    )
+    (property "Value" "AD7490BCPZ" (id 1) (at 162.56 104.14 0)
+      (effects (font (size 1.524 1.524)))
+    )
+    (property "Footprint" "CP_32_2_ADI" (id 2) (at 129.54 111.76 0)
+      (effects (font (size 1.27 1.27) italic) hide)
+    )
+    (property "Datasheet" "AD7490BCPZ" (id 3) (at 129.54 111.76 0)
+      (effects (font (size 1.27 1.27) italic) hide)
+    )
+    (pin "1")
+    (pin "10")
+    (pin "11")
+    (pin "12")
+    (pin "13")
+    (pin "14")
+    (pin "15")
+    (pin "16")
+    (pin "17")
+    (pin "18")
+    (pin "19")
+    (pin "2")
+    (pin "20")
+    (pin "21")
+    (pin "22")
+    (pin "23")
+    (pin "24")
+    (pin "25")
+    (pin "26")
+    (pin "27")
+    (pin "28")
+    (pin "29")
+    (pin "3")
+    (pin "30")
+    (pin "31")
+    (pin "32")
+    (pin "33")
+    (pin "4")
+    (pin "5")
+    (pin "6")
+    (pin "7")
+    (pin "8")
+    (pin "9")
+  )
 )

Commit message: wip
Parts:
- removed U2: CD74HC4067M, Package_SO:SOIC-24W_7.5x15.4mm_P1.27mm, symbol 74xx:CD74HC4067M
Connections:
- net +3V3: now also U?.25 (EP)
- net SCL: now reaches U?.19 (SCL)
- net SDA: now reaches U?.20 (SDA)
- net *INT: now reaches U?.22 (*INT)
- net RESET_IOEXP: now reaches U?.24 (*RESET)
Other:
- note added: "I2C interface for IO expender"
- moved on the sheet: U?

Commit message: schematic finished
Parts:
- removed J3: Conn_02x10_MountingPin, Connector_PinHeader_2.54mm:PinHeader_2x10_P2.54mm_Vertical_SMD, symbol Connector_Generic_MountingPin:Conn_01x20_MountingPin
- added C29, C30, C31, C32, C33, C36: 0.1uF, symbol Device:C_Small
- added C34, C35: 10uF, symbol Device:C_Small
- added J3, J4, J5: Conn_02x12_Counter_Clockwise_MountingPin, symbol Connector_Generic_MountingPin:Conn_02x12_Counter_Clockwise_MountingPin
- added R20: 25, symbol Device:R_US
Connections:
- net *INT: now also R20.2
- net +3V3: now also U?.15 (VDRIVE), C33.1, C34.1, J3.1 (Pin_1), R20.1
- net GNDREF: now also U?.18 (ADDR), U?.33, C29.2, C30.2, C31.2, C32.2, C33.2, C34.2, C35.2, C36.2, J3.15 (Pin_15), J3.16 (Pin_16), J3.17 (Pin_17), J3.24 (Pin_24), J3.8 (Pin_8), J3.MP (MountPin), J4.10 (Pin_10), J4.12 (Pin_12), J4.13 (Pin_13), J4.15 (Pin_15), J4.18 (Pin_18), J4.20 (Pin_20), J4.22 (Pin_22), J4.3 (Pin_3), J4.5 (Pin_5), J4.7 (Pin_7), J4.MP (MountPin), J5.10 (Pin_10), J5.15 (Pin_15), J5.17 (Pin_17), J5.19 (Pin_19), J5.2 (Pin_2), J5.21 (Pin_21), J5.23 (Pin_23), J5.4 (Pin_4), J5.6 (Pin_6), J5.8 (Pin_8), J5.MP (MountPin)
- net SPI3_CLK: now also U?.14 (SCLK), J3.11 (Pin_11), J3.21 (Pin_21), J3.4 (Pin_4)
- net SPI3_CS0: now also U?.18 (CS*)
- net SPI3_CS1: now also J3.5 (Pin_5)
- net SPI3_CS2: now also J3.12 (Pin_12)
- net SPI3_CS3: now also J3.20 (Pin_20)
- net SPI3_MISO: now also U?.13 (DOUT), J3.10 (Pin_10), J3.22 (Pin_22), J3.3 (Pin_3)
- net SPI3_MOSI: now also U?.17 (DIN), J3.2 (Pin_2), J3.23 (Pin_23), J3.9 (Pin_9)
- net OUTPUT_IOEXP_0: now reaches U?.1 (P0_0)
- net OUTPUT_IOEXP_0: now also J5.18 (Pin_18)
- net INPUT_IOEXP_0: now reaches U?.10 (P1_0)
- net INPUT_IOEXP_0: now also J5.7 (Pin_7)
- net INPUT_IOEXP_1: now reaches U?.11 (P1_1)
- net INPUT_IOEXP_1: now also J5.1 (Pin_1)
- net INPUT_IOEXP_2: now reaches U?.12 (P1_2)
- net INPUT_IOEXP_2: now also J4.24 (Pin_24)
- net INPUT_IOEXP_3: now reaches U?.13 (P1_3)
- net INPUT_IOEXP_3: now also J4.8 (Pin_8)
- net INPUT_IOEXP_4: now reaches U?.14 (P1_4)
- net INPUT_IOEXP_4: now also J4.2 (Pin_2)
- net INPUT_IOEXP_5: now reaches U?.15 (P1_5)
- net INPUT_IOEXP_5: now also J3.6 (Pin_6)
- net INPUT_IOEXP_6: now reaches U?.16 (P1_6)
- net INPUT_IOEXP_6: now also J3.14 (Pin_14)
- net INPUT_IOEXP_7: now reaches U?.17 (P1_7)
- net INPUT_IOEXP_7: now also J3.19 (Pin_19)
- net OUTPUT_IOEXP_1: now reaches U?.2 (P0_1)
- net OUTPUT_IOEXP_1: now also J5.24 (Pin_24)
- net OUTPUT_IOEXP_2: now reaches U?.3 (P0_2)
- net OUTPUT_IOEXP_2: now also J4.23 (Pin_23)
- net OUTPUT_IOEXP_3: now reaches U?.4 (P0_3)
- net OUTPUT_IOEXP_3: now also J4.17 (Pin_17)
- net OUTPUT_IOEXP_4: now reaches U?.5 (P0_4)
- net OUTPUT_IOEXP_4: now also J4.1 (Pin_1)
- net OUTPUT_IOEXP_5: now reaches U?.6 (P0_5)
- net OUTPUT_IOEXP_5: now also J3.7 (Pin_7)
- net OUTPUT_IOEXP_6: now reaches U?.7 (P0_6)
- net OUTPUT_IOEXP_6: now also J3.13 (Pin_13)
- net OUTPUT_IOEXP_7: now reaches U?.8 (P0_7)
- net OUTPUT_IOEXP_7: now also J3.18 (Pin_18)
- net ADC_BOARD_IN_1: now reaches U?.10 (VIN1)
- net ADC_BOARD_IN_1: now also J5.11 (Pin_11)
- net ADC_BOARD_IN_0: now reaches U?.11 (VIN0)
- net ADC_BOARD_IN_0: now also J5.14 (Pin_14)
- net at U?.12 (AGND): now also C30.1
- net at U?.19 (AGND): now also C29.1
- net ADC_BOARD_IN_8: now reaches U?.2 (VIN8)
- net ADC_BOARD_IN_8: now also J4.21 (Pin_21)
- net +3.3VA: now reaches U?.20 (VDD)
- net +3.3VA: now also C35.1, C36.1
- net VREF_IN: now reaches U?.21 (REFIN)
- net VREF_IN: now also C32.1
- net at U?.22 (AGND): now also C31.1
- net ADC_BOARD_IN_15: now reaches U?.24 (VIN15)
- net ADC_BOARD_IN_15: now also J4.4 (Pin_4)
- net ADC_BOARD_IN_14: now reaches U?.26 (VIN14)
- net ADC_BOARD_IN_14: now also J4.6 (Pin_6)
- net ADC_BOARD_IN_13: now reaches U?.27 (VIN13)
- net ADC_BOARD_IN_13: now also J4.9 (Pin_9)
- net ADC_BOARD_IN_12: now reaches U?.28 (VIN12)
- net ADC_BOARD_IN_12: now also J4.11 (Pin_11)
- net ADC_BOARD_IN_11: now reaches U?.29 (VIN11)
- net ADC_BOARD_IN_11: now also J4.14 (Pin_14)
- net ADC_BOARD_IN_7: now reaches U?.3 (VIN7)
- net ADC_BOARD_IN_7: now also J5.3 (Pin_3)
- net ADC_BOARD_IN_10: now reaches U?.30 (VIN10)
- net ADC_BOARD_IN_10: now also J4.16 (Pin_16)
- net ADC_BOARD_IN_9: now reaches U?.31 (VIN9)
- net ADC_BOARD_IN_9: now also J4.19 (Pin_19)
- net ADC_BOARD_IN_6: now reaches U?.4 (VIN6)
- net ADC_BOARD_IN_6: now also J5.22 (Pin_22)
- net ADC_BOARD_IN_5: now reaches U?.5 (VIN5)
- net ADC_BOARD_IN_5: now also J5.5 (Pin_5)
- net ADC_BOARD_IN_4: now reaches U?.6 (VIN4)
- net ADC_BOARD_IN_4: now also J5.20 (Pin_20)
- net ADC_BOARD_IN_3: now reaches U?.7 (VIN3)
- net ADC_BOARD_IN_3: now also J5.9 (Pin_9)
- net ADC_BOARD_IN_2: now reaches U?.9 (VIN2)
- net ADC_BOARD_IN_2: now also J5.16 (Pin_16)
- no-connect marks 0 -> 6
Other:
- note added: "ADC AND IO EXPENDER BRANCH OUT"
- note added: "ADC multi-source programmable"
- note added: "ADDR : 0b"
- note added: "IO EXPENDER"
- note added: "SPI communication branch out"
- note added: "VDD = 3 V, fSCLK = 16 MHz"
- note added: "max output current = 160 mA"
- note removed: "Probes connector branch out"
- moved on the sheet: U?

Commit message: Schematic update
Parts:
- C29, C30, C31, C32, C33, C36: footprint (none) -> Capacitor_SMD:C_1206_3216Metric_Pad1.33x1.80mm_HandSolder; MPN (none) -> CC1206KRX7R9BB104; Supplier Link (none) -> https://www.digikey.ca/en/products/detail/yageo/CC1206KRX7R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
- C34, C35: footprint (none) -> Capacitor_SMD:C_1206_3216Metric_Pad1.33x1.80mm_HandSolder; MPN (none) -> CL31B106KAHNNNE; Supplier Link (none) -> https://www.digikey.ca/en/products/detail/samsung-electro-m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
- gave numbers to parts that had none: 2
Changed lines of the file:
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@@
   (symbol (lib_id "PI4IOE5V6416ZDEX:PI4IOE5V6416ZDEX") (at 92.71 38.1 0) (unit 1)
     (in_bom yes) (on_board yes) (dnp no) (fields_autoplaced)
-    (property "Reference" "U?" (at 120.65 26.67 0)
+    (property "Reference" "U10" (at 120.65 26.67 0)
       (effects (font (size 1.524 1.524)))
     )
@@
       (project "Synaps_PCB_2021"
         (path "/e63e39d7-6ac0-4ffd-8aa3-1841a4541b55/00000000-0000-0000-0000-0000604b51e6"
-          (reference "U?") (unit 1)
+          (reference "U10") (unit 1)
         )
       )
@@
       (effects (font (size 1.27 1.27)) (justify left))
     )
-    (property "Footprint" "" (at 142.24 168.91 0)
-      (effects (font (size 1.27 1.27)) hide)
-    )
-    (property "Datasheet" "~" (at 142.24 168.91 0)
+    (property "Footprint" "Capacitor_SMD:C_1206_3216Metric_Pad1.33x1.80mm_HandSolder" (at 142.24 168.91 0)
+      (effects (font (size 1.27 1.27)) hide)
+    )
+    (property "Datasheet" "https://media.digikey.com/pdf/Data%20Sheets/Samsung%20PDFs/CL31B106KAHNNNE_Spec.pdf" (at 142.24 168.91 0)
+      (effects (font (size 1.27 1.27)) hide)
+    )
+    (property "MPN" "CL31B106KAHNNNE" (at 142.24 168.91 0)
+      (effects (font (size 1.27 1.27)) hide)
+    )
+    (property "Supplier Link" "https://www.digikey.ca/en/products/detail/samsung-electro-mechanics/CL31B106KAHNNNE/3887462" (at 142.24 168.91 0)
       (effects (font (size 1.27 1.27)) hide)
     )
@@
       (effects (font (size 1.27 1.27)) (justify left))
     )
-    (property "Footprint" "" (at 34.29 171.45 0)
-      (effects (font (size 1.27 1.27)) hide)
-    )
-    (property "Datasheet" "~" (at 34.29 171.45 0)
+    (property "Footprint" "Capacitor_SMD:C_1206_3216Metric_Pad1.33x1.80mm_HandSolder" (at 34.29 171.45 0)
+      (effects (font (size 1.27 1.27)) hide)
+    )
+    (property "Datasheet" "https://media.digikey.com/pdf/Data%20Sheets/Samsung%20PDFs/CL31B106KAHNNNE_Spec.pdf" (at 34.29 171.45 0)
+      (effects (font (size 1.27 1.27)) hide)
+    )
+    (property "MPN" "CL31B106KAHNNNE" (at 34.29 171.45 0)
+      (effects (font (size 1.27 1.27)) hide)
+    )
+    (property "Supplier Link" "https://www.digikey.ca/en/products/detail/samsung-electro-mechanics/CL31B106KAHNNNE/3887462" (at 34.29 171.45 0)
       (effects (font (size 1.27 1.27)) hide)
     )
@@
       (effects (font (size 1.27 1.27)) (justify left))
     )
-    (property "Footprint" "" (at 133.35 168.91 0)
-      (effects (font (size 1.27 1.27)) hide)
-    )
-    (property "Datasheet" "~" (at 133.35 168.91 0)
+    (property "Footprint" "Capacitor_SMD:C_1206_3216Metric_Pad1.33x1.80mm_HandSolder" (at 133.35 168.91 0)
+      (effects (font (size 1.27 1.27)) hide)
+    )
+    (property "Datasheet" "https://www.yageo.com/upload/media/product/productsearch/datasheet/mlcc/UPY-GPHC_X7R_6.3V-to-50V_20.pdf" (at 133.35 168.91 0)
+      (effects (font (size 1.27 1.27)) hide)
+    )
+    (property "MPN" "CC1206KRX7R9BB104" (at 133.35 168.91 0)
+      (effects (font (size 1.27 1.27)) hide)
+    )
+    (property "Supplier Link" "https://www.digikey.ca/en/products/detail/yageo/CC1206KRX7R9BB104/302913" (at 133.35 168.91 0)
       (effects (font (size 1.27 1.27)) hide)
     )
@@
   (symbol (lib_id "power:+3.3V") (at 156.21 38.1 0) (unit 1)
     (in_bom yes) (on_board yes) (dnp no) (fields_autoplaced)
-    (property "Reference" "#PWR?" (at 156.21 41.91 0)
+    (property "Reference" "#PWR0108" (at 156.21 41.91 0)
       (effects (font (size 1.27 1.27)) hide)
     )
@@
       (project "Synaps_PCB_2021"
         (path "/e63e39d7-6ac0-4ffd-8aa3-1841a4541b55/00000000-0000-0000-0000-0000604b51e6"
-          (reference "#PWR?") (unit 1)
+          (reference "#PWR0108") (unit 1)
         )
       )
@@
       (effects (font (size 1.27 1.27)) (justify left))
     )
-    (property "Footprint" "" (at 127 179.07 0)
-      (effects (font (size 1.27 1.27)) hide)
-    )
-    (property "Datasheet" "~" (at 127 179.07 0)
+    (property "Footprint" "Capacitor_SMD:C_1206_3216Metric_Pad1.33x1.80mm_HandSolder" (at 127 179.07 0)
+      (effects (font (size 1.27 1.27)) hide)
+    )
+    (property "Datasheet" "https://www.yageo.com/upload/media/product/productsearch/datasheet/mlcc/UPY-GPHC_X7R_6.3V-to-50V_20.pdf" (at 127 179.07 0)
+      (effects (font (size 1.27 1.27)) hide)
+    )
+    (property "MPN" "CC1206KRX7R9BB104" (at 127 179.07 0)
+      (effects (font (size 1.27 1.27)) hide)
+    )
+    (property "Supplier Link" "https://www.digikey.ca/en/products/detail/yageo/CC1206KRX7R9BB104/302913" (at 127 179.07 0)
       (effects (font (size 1.27 1.27)) hide)
     )
@@
       (effects (font (size 1.27 1.27)) (justify left))
     )
-    (property "Footprint" "" (at 149.86 166.37 0)
-      (effects (font (size 1.27 1.27)) hide)
-    )
-    (property "Datasheet" "~" (at 149.86 166.37 0)
+    (property "Footprint" "Capacitor_SMD:C_1206_3216Metric_Pad1.33x1.80mm_HandSolder" (at 149.86 166.37 0)
+      (effects (font (size 1.27 1.27)) hide)
+    )
+    (property "Datasheet" "https://www.yageo.com/upload/media/product/productsearch/datasheet/mlcc/UPY-GPHC_X7R_6.3V-to-50V_20.pdf" (at 149.86 166.37 0)
+      (effects (font (size 1.27 1.27)) hide)
+    )
+    (property "MPN" "CC1206KRX7R9BB104" (at 149.86 166.37 0)
+      (effects (font (size 1.27 1.27)) hide)
+    )
+    (property "Supplier Link" "https://www.digikey.ca/en/products/detail/yageo/CC1206KRX7R9BB104/302913" (at 149.86 166.37 0)
       (effects (font (size 1.27 1.27)) hide)
     )
@@
       (effects (font (size 1.27 1.27)) (justify left))
     )
-    (property "Footprint" "" (at 41.91 171.45 0)
-      (effects (font (size 1.27 1.27)) hide)
-    )
-    (property "Datasheet" "~" (at 41.91 171.45 0)
+    (property "Footprint" "Capacitor_SMD:C_1206_3216Metric_Pad1.33x1.80mm_HandSolder" (at 41.91 171.45 0)
+      (effects (font (size 1.27 1.27)) hide)
+    )
+    (property "Datasheet" "https://www.yageo.com/upload/media/product/productsearch/datasheet/mlcc/UPY-GPHC_X7R_6.3V-to-50V_20.pdf" (at 41.91 171.45 0)
+      (effects (font (size 1.27 1.27)) hide)
+    )
+    (property "MPN" "CC1206KRX7R9BB104" (at 41.91 171.45 0)
+      (effects (font (size 1.27 1.27)) hide)
+    )
+    (property "Supplier Link" "https://www.digikey.ca/en/products/detail/yageo/CC1206KRX7R9BB104/302913" (at 41.91 171.45 0)
       (effects (font (size 1.27 1.27)) hide)
     )
@@
       (effects (font (size 1.27 1.27)) (justify left))
     )
-    (property "Footprint" "" (at 26.67 163.83 0)
-      (effects (font (size 1.27 1.27)) hide)
-    )
-    (property "Datasheet" "~" (at 26.67 163.83 0)
+    (property "Footprint" "Capacitor_SMD:C_1206_3216Metric_Pad1.33x1.80mm_HandSolder" (at 26.67 163.83 0)
+      (effects (font (size 1.27 1.27)) hide)
+    )
+    (property "Datasheet" "https://www.yageo.com/upload/media/product/productsearch/datasheet/mlcc/UPY-GPHC_X7R_6.3V-to-50V_20.pdf" (at 26.67 163.83 0)
+      (effects (font (size 1.27 1.27)) hide)
+    )
+    (property "MPN" "CC1206KRX7R9BB104" (at 26.67 163.83 0)
+      (effects (font (size 1.27 1.27)) hide)
+    )
+    (property "Supplier Link" "https://www.digikey.ca/en/products/detail/yageo/CC1206KRX7R9BB104/302913" (at 26.67 163.83 0)
       (effects (font (size 1.27 1.27)) hide)
     )
@@
       (effects (font (size 1.27 1.27)) (justify left))
     )
-    (property "Footprint" "" (at 157.48 163.83 0)
-      (effects (font (size 1.27 1.27)) hide)
-    )
-    (property "Datasheet" "~" (at 157.48 163.83 0)
+    (property "Footprint" "Capacitor_SMD:C_1206_3216Metric_Pad1.33x1.80mm_HandSolder" (at 157.48 163.83 0)
+      (effects (font (size 1.27 1.27)) hide)
+    )
+    (property "Datasheet" "https://www.yageo.com/upload/media/product/productsearch/datasheet/mlcc/UPY-GPHC_X7R_6.3V-to-50V_20.pdf" (at 157.48 163.83 0)
+      (effects (font (size 1.27 1.27)) hide)
+    )
+    (property "MPN" "CC1206KRX7R9BB104" (at 157.48 163.83 0)
+      (effects (font (size 1.27 1.27)) hide)
+    )
+    (property "Supplier Link" "https://www.digikey.ca/en/products/detail/yageo/CC1206KRX7R9BB104/302913" (at 157.48 163.83 0)
       (effects (font (size 1.27 1.27)) hide)
     )
@@
   (symbol (lib_id "AD7490BCPZ:AD7490BCPZ") (at 46.99 133.35 0) (unit 1)
     (in_bom yes) (on_board yes) (dnp no) (fields_autoplaced)
-    (property "Reference" "U?" (at 80.01 121.92 0)
+    (property "Reference" "U2" (at 80.01 121.92 0)
       (effects (font (size 1.524 1.524)))
     )
@@
       (project "Synaps_PCB_2021"
         (path "/e63e39d7-6ac0-4ffd-8aa3-1841a4541b55/00000000-0000-0000-0000-0000604b51e6"
-          (reference "U?") (unit 1)
-        )
-      )
+          (reference "U2") (unit 1)
+        )
+      )
