File: KiCAD_project_folder/Synaps_PCB_2021/batcharg.kicad_sch (KiCad schematic)
At the start: 15 parts

Commit message: wip
Parts:
- added BT? (x2): Battery_Cell, Battery:BatteryHolder_Keystone_2462_2xAA, symbol Device:Battery_Cell
- added C20: 22uF, symbol Device:C
- added C? (x3): 0.1uF, symbol Device:C
- added R? (x3): 1000, symbol Device:R_US
- added TP?: Batt_plus, symbol Connector:TestPoint
- added TP?: Batt_minus, symbol Connector:TestPoint
- C16: renamed from C?; value C -> 1uF
- C17: renamed from C?; value C -> 22uF
- C18: renamed from C?; value C -> 100nF
- C19: renamed from C?; value C -> 0.47uF
- L6: renamed from L?; value INDUCTOR -> 6.8uH
- R11: renamed from R?; value R_US -> 50m; Description  (none) -> RS1
- gave numbers to parts that had none: 9
Connections:
- net GNDREF: now also R10.2, U7.7 (VSS), U7.9 (PAD), BT?.2 (-), C20.2, C?.1, C?.2, TP?.1
- net at U7.1 (VDD): now also C?.2, R?.1
- net at U7.2 (V5): now also U7.3 (V4), U7.4 (V3), U7.5 (V2), C?.1, R?.1
- net at U7.6 (V1): now also C?.1, C?.2, R?.1
- net BATT_OVERVOLTAGE_OUT: now reaches U7.8 (OUT)
- net BATT_CHARGING renamed V_BAT
- net V_BAT: now also BT?.1 (+), C20.1, R?.2, R?.2, TP?.1
- new net: BT?.1 (+), BT?.2 (-), R?.2
Other:
- moved on the sheet: U7

Commit message: Schematic update
Parts:
- C16: footprint (none) -> Capacitor_SMD:C_1206_3216Metric_Pad1.33x1.80mm_HandSolder; MPN (none) -> GCM31MR71H105KA55L; Supplier Link (none) -> https://www.digikey.ca/en/products/detail/murata-electronic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
- C37, C38, C39: renamed from C?; footprint (none) -> Capacitor_SMD:C_1206_3216Metric_Pad1.33x1.80mm_HandSolder; MPN (none) -> CC1206KRX7R9BB104; Supplier Link (none) -> https://www.digikey.ca/en/products/detail/yageo/CC1206KRX7R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
- R5: value R_US -> 1k NTC; footprint (none) -> LED_SMD:LED_0805_2012Metric_Pad1.15x1.40mm_HandSolder; MPN (none) -> B57421V2102J062; Supplier Link (none) -> https://www.digikey.ca/fr/products/detail/epcos-tdk-electro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
- R9: value R_US -> 10K
- gave numbers to parts that had none: 7
