File: KiCAD_project_folder/Synaps_PCB_2021/voltreg.kicad_sch (KiCad schematic)
At the start: 12 parts

Commit message: wip
Parts:
- C21, C22, C23, C24: renamed from C?; value 22u -> 22uF
- C25, C26: renamed from C?; value 10u -> 10uF
- C27, C28: renamed from C?; value 100n -> 100nF
- gave numbers to parts that had none: 4
Changed lines of the file:
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@@
   (symbol (lib_id "Device:C") (at 111.76 107.95 0) (unit 1)
     (in_bom yes) (on_board yes)
-    (property "Reference" "C?" (id 0) (at 113.03 105.41 0)
-      (effects (font (size 1.27 1.27)) (justify left))
-    )
-    (property "Value" "22u" (id 1) (at 113.03 110.49 0)
+    (property "Reference" "C24" (id 0) (at 113.03 105.41 0)
+      (effects (font (size 1.27 1.27)) (justify left))
+    )
+    (property "Value" "22uF" (id 1) (at 113.03 110.49 0)
       (effects (font (size 1.27 1.27)) (justify left))
     )
@@
   (symbol (lib_id "Device:C") (at 162.56 107.95 0) (unit 1)
     (in_bom yes) (on_board yes)
-    (property "Reference" "C?" (id 0) (at 163.83 104.14 0)
-      (effects (font (size 1.27 1.27)) (justify left))
-    )
-    (property "Value" "100n" (id 1) (at 163.83 111.76 0)
+    (property "Reference" "C28" (id 0) (at 163.83 104.14 0)
+      (effects (font (size 1.27 1.27)) (justify left))
+    )
+    (property "Value" "100nF" (id 1) (at 163.83 111.76 0)
       (effects (font (size 1.27 1.27)) (justify left))
     )
@@
   (symbol (lib_id "power:GNDREF") (at 106.68 134.62 0) (unit 1)
     (in_bom yes) (on_board yes) (fields_autoplaced)
-    (property "Reference" "#PWR?" (id 0) (at 106.68 140.97 0)
+    (property "Reference" "#PWR061" (id 0) (at 106.68 140.97 0)
       (effects (font (size 1.27 1.27)) hide)
     )
@@
   (symbol (lib_id "Device:C") (at 111.76 41.91 0) (unit 1)
     (in_bom yes) (on_board yes)
-    (property "Reference" "C?" (id 0) (at 113.03 39.37 0)
-      (effects (font (size 1.27 1.27)) (justify left))
-    )
-    (property "Value" "22u" (id 1) (at 113.03 44.45 0)
+    (property "Reference" "C23" (id 0) (at 113.03 39.37 0)
+      (effects (font (size 1.27 1.27)) (justify left))
+    )
+    (property "Value" "22uF" (id 1) (at 113.03 44.45 0)
       (effects (font (size 1.27 1.27)) (justify left))
     )
@@
   (symbol (lib_id "AP63203WU-7:AP63203WU-7") (at 119.38 46.99 0) (unit 1)
     (in_bom yes) (on_board yes) (fields_autoplaced)
-    (property "Reference" "U?" (id 0) (at 139.7 35.56 0)
+    (property "Reference" "U8" (id 0) (at 139.7 35.56 0)
       (effects (font (size 1.524 1.524)))
     )
@@
   (symbol (lib_id "Device:C") (at 162.56 41.91 0) (unit 1)
     (in_bom yes) (on_board yes)
-    (property "Reference" "C?" (id 0) (at 163.83 38.1 0)
-      (effects (font (size 1.27 1.27)) (justify left))
-    )
-    (property "Value" "100n" (id 1) (at 163.83 45.72 0)
+    (property "Reference" "C27" (id 0) (at 163.83 38.1 0)
+      (effects (font (size 1.27 1.27)) (justify left))
+    )
+    (property "Value" "100nF" (id 1) (at 163.83 45.72 0)
       (effects (font (size 1.27 1.27)) (justify left))
     )
@@
   (symbol (lib_id "power:GNDREF") (at 114.3 60.96 0) (unit 1)
     (in_bom yes) (on_board yes) (fields_autoplaced)
-    (property "Reference" "#PWR?" (id 0) (at 114.3 67.31 0)
+    (property "Reference" "#PWR062" (id 0) (at 114.3 67.31 0)
       (effects (font (size 1.27 1.27)) hide)
     )
@@
   (symbol (lib_id "power:GNDREF") (at 114.3 127 0) (unit 1)
     (in_bom yes) (on_board yes) (fields_autoplaced)
-    (property "Reference" "#PWR?" (id 0) (at 114.3 133.35 0)
+    (property "Reference" "#PWR063" (id 0) (at 114.3 133.35 0)
       (effects (font (size 1.27 1.27)) hide)
     )
@@
   (symbol (lib_id "Device:C") (at 101.6 41.91 0) (unit 1)
     (in_bom yes) (on_board yes)
-    (property "Reference" "C?" (id 0) (at 102.87 39.37 0)
-      (effects (font (size 1.27 1.27)) (justify left))
-    )
-    (property "Value" "22u" (id 1) (at 102.87 44.45 0)
+    (property "Reference" "C21" (id 0) (at 102.87 39.37 0)
+      (effects (font (size 1.27 1.27)) (justify left))
+    )
+    (property "Value" "22uF" (id 1) (at 102.87 44.45 0)
       (effects (font (size 1.27 1.27)) (justify left))
     )
@@
   (symbol (lib_id "pspice:INDUCTOR") (at 139.7 99.06 0) (unit 1)
     (in_bom yes) (on_board yes) (fields_autoplaced)
-    (property "Reference" "L?" (id 0) (at 139.7 92.71 0))
+    (property "Reference" "L8" (id 0) (at 139.7 92.71 0))
     (property "Value" "4.7u" (id 1) (at 139.7 95.25 0))
     (property "Footprint" "" (id 2) (at 139.7 99.06 0)
@@
   (symbol (lib_id "pspice:INDUCTOR") (at 139.7 33.02 0) (unit 1)
     (in_bom yes) (on_board yes) (fields_autoplaced)
-    (property "Reference" "L?" (id 0) (at 139.7 26.67 0))
+    (property "Reference" "L7" (id 0) (at 139.7 26.67 0))
     (property "Value" "4.7u" (id 1) (at 139.7 29.21 0))
     (property "Footprint" "" (id 2) (at 139.7 33.02 0)
@@
   (symbol (lib_id "Device:C") (at 114.3 121.92 0) (unit 1)
     (in_bom yes) (on_board yes) (fields_autoplaced)
-    (property "Reference" "C?" (id 0) (at 118.11 120.6499 0)
-      (effects (font (size 1.27 1.27)) (justify left))
-    )
-    (property "Value" "10u" (id 1) (at 118.11 123.1899 0)
+    (property "Reference" "C26" (id 0) (at 118.11 120.6499 0)
+      (effects (font (size 1.27 1.27)) (justify left))
+    )
+    (property "Value" "10uF" (id 1) (at 118.11 123.1899 0)
       (effects (font (size 1.27 1.27)) (justify left))
     )
@@
   (symbol (lib_id "Device:C") (at 101.6 107.95 0) (unit 1)
     (in_bom yes) (on_board yes)
-    (property "Reference" "C?" (id 0) (at 102.87 105.41 0)
-      (effects (font (size 1.27 1.27)) (justify left))
-    )
-    (property "Value" "22u" (id 1) (at 102.87 110.49 0)
+    (property "Reference" "C22" (id 0) (at 102.87 105.41 0)
+      (effects (font (size 1.27 1.27)) (justify left))
+    )
+    (property "Value" "22uF" (id 1) (at 102.87 110.49 0)
       (effects (font (size 1.27 1.27)) (justify left))
     )
@@
   (symbol (lib_id "power:GNDREF") (at 106.68 68.58 0) (unit 1)
     (in_bom yes) (on_board yes) (fields_autoplaced)
-    (property "Reference" "#PWR?" (id 0) (at 106.68 74.93 0)
+    (property "Reference" "#PWR060" (id 0) (at 106.68 74.93 0)
       (effects (font (size 1.27 1.27)) hide)
     )
@@
   (symbol (lib_id "Device:C") (at 114.3 55.88 0) (unit 1)
     (in_bom yes) (on_board yes) (fields_autoplaced)
-    (property "Reference" "C?" (id 0) (at 118.11 54.6099 0)
-      (effects (font (size 1.27 1.27)) (justify left))
-    )
-    (property "Value" "10u" (id 1) (at 118.11 57.1499 0)
+    (property "Reference" "C25" (id 0) (at 118.11 54.6099 0)
+      (effects (font (size 1.27 1.27)) (justify left))
+    )
+    (property "Value" "10uF" (id 1) (at 118.11 57.1499 0)
       (effects (font (size 1.27 1.27)) (justify left))
     )
@@
   (symbol (lib_id "AP63205WU-7:AP63205WU-7") (at 119.38 113.03 0) (unit 1)
     (in_bom yes) (on_board yes) (fields_autoplaced)
-    (property "Reference" "U?" (id 0) (at 139.7 101.6 0)
+    (property "Reference" "U9" (id 0) (at 139.7 101.6 0)
       (effects (font (size 1.524 1.524)))
     )

Commit message: Schematic update
Parts:
- C25, C26: footprint (none) -> Capacitor_SMD:C_1206_3216Metric_Pad1.33x1.80mm_HandSolder; MPN (none) -> CL31B106KAHNNNE; Supplier Link (none) -> https://www.digikey.ca/en/products/detail/samsung-electro-m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
- L7, L8: value 4.7u -> 4.7uH
Changed lines of the file:
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@@
       (effects (font (size 1.27 1.27)))
     )
-    (property "Value" "4.7u" (at 139.7 95.25 0)
+    (property "Value" "4.7uH" (at 139.7 95.25 0)
       (effects (font (size 1.27 1.27)))
     )
@@
       (effects (font (size 1.27 1.27)))
     )
-    (property "Value" "4.7u" (at 139.7 29.21 0)
+    (property "Value" "4.7uH" (at 139.7 29.21 0)
       (effects (font (size 1.27 1.27)))
     )
@@
       (effects (font (size 1.27 1.27)) (justify left))
     )
-    (property "Footprint" "" (at 115.2652 125.73 0)
+    (property "Footprint" "Capacitor_SMD:C_1206_3216Metric_Pad1.33x1.80mm_HandSolder" (at 115.2652 125.73 0)
       (effects (font (size 1.27 1.27)) hide)
     )
-    (property "Datasheet" "~" (at 114.3 121.92 0)
+    (property "Datasheet" "https://media.digikey.com/pdf/Data%20Sheets/Samsung%20PDFs/CL31B106KAHNNNE_Spec.pdf" (at 114.3 121.92 0)
+      (effects (font (size 1.27 1.27)) hide)
+    )
+    (property "MPN" "CL31B106KAHNNNE" (at 114.3 121.92 0)
+      (effects (font (size 1.27 1.27)) hide)
+    )
+    (property "Supplier Link" "https://www.digikey.ca/en/products/detail/samsung-electro-mechanics/CL31B106KAHNNNE/3887462" (at 114.3 121.92 0)
       (effects (font (size 1.27 1.27)) hide)
     )
@@
       (effects (font (size 1.27 1.27)) (justify left))
     )
-    (property "Footprint" "" (at 115.2652 59.69 0)
+    (property "Footprint" "Capacitor_SMD:C_1206_3216Metric_Pad1.33x1.80mm_HandSolder" (at 115.2652 59.69 0)
       (effects (font (size 1.27 1.27)) hide)
     )
-    (property "Datasheet" "~" (at 114.3 55.88 0)
+    (property "Datasheet" "https://media.digikey.com/pdf/Data%20Sheets/Samsung%20PDFs/CL31B106KAHNNNE_Spec.pdf" (at 114.3 55.88 0)
       (effects (font (size 1.27 1.27)) hide)
     )
+    (property "MPN" "CL31B106KAHNNNE" (at 114.3 55.88 0)
+      (effects (font (size 1.27 1.27)) hide)
+    )
+    (property "Supplier Link" "https://www.digikey.ca/en/products/detail/samsung-electro-mechanics/CL31B106KAHNNNE/3887462" (at 114.3 55.88 0)
+      (effects (font (size 1.27 1.27)) hide)
+    )
