File: KiCAD_project_folder/Probe_PCB/high_pass_filter.kicad_sch (KiCad schematic)
At the start: 0 parts

Commit message: added schematic for filters and amplifier
Parts:
- added C2: 100 uF, symbol Device:C
- added R1: 10K, symbol Device:R_US
- added U1: OPA1622, Package_SON:Texas_S-PVSON-N10, symbol Amplifier_Audio:OPA1622
Connections:
- new net: C2.1, R1.2, U1.1 (+)
- new net GNDREF: R1.1
- new net Vin_HIGHPASS: C2.2
- new net Vout_HIGHPASS: U1.10 (-), U1.9
Other:
- note added: "RC network, low-pass, R = 10K, C = 99.99 uF and fc = 0.16 Hz"
Changed lines of the file:
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@@
 (kicad_sch (version 20230121) (generator eeschema)
   (paper "A4")
+  (junction (at 141.605 102.87) (diameter 0) (color 0 0 0 0)
+  )
+  (junction (at 113.665 83.82) (diameter 0) (color 0 0 0 0)
+  )
+  (junction (at 141.605 81.28) (diameter 0) (color 0 0 0 0)
+  )
+  (wire (pts (xy 141.605 81.28) (xy 149.225 81.28))
+    (stroke (width 0) (type default))
+  )
+  (wire (pts (xy 141.605 102.87) (xy 165.735 102.87))
+    (stroke (width 0) (type default))
+  )
+  (wire (pts (xy 108.585 102.87) (xy 141.605 102.87))
+    (stroke (width 0) (type default))
+  )
+  (wire (pts (xy 156.845 81.28) (xy 165.735 81.28))
+    (stroke (width 0) (type default))
+  )
+  (wire (pts (xy 128.905 81.28) (xy 141.605 81.28))
+    (stroke (width 0) (type default))
+  )
+  (wire (pts (xy 132.08 86.36) (xy 132.08 92.71))
+    (stroke (width 0) (type default))
+  )
+  (wire (pts (xy 141.605 92.71) (xy 141.605 102.87))
+    (stroke (width 0) (type default))
+  )
+  (wire (pts (xy 132.08 86.36) (xy 128.905 86.36))
+    (stroke (width 0) (type default))
+  )
+  (wire (pts (xy 108.585 83.82) (xy 113.665 83.82))
+    (stroke (width 0) (type default))
+  )
+  (wire (pts (xy 113.665 92.71) (xy 113.665 83.82))
+    (stroke (width 0) (type default))
+  )
+  (wire (pts (xy 113.665 92.71) (xy 132.08 92.71))
+    (stroke (width 0) (type default))
+  )
+  (wire (pts (xy 141.605 81.28) (xy 141.605 85.09))
+    (stroke (width 0) (type default))
+  )
+  (rectangle (start 71.12 55.88) (end 215.9 135.89)
+    (stroke (width 0) (type default))
+    (fill (type none))
+  )
+  (text "RC network, low-pass, R = 10K, C = 99.99 uF and fc = 0.16 Hz"
+    (at 71.12 53.34 0)
+    (effects (font (size 1.27 1.27)) (justify left bottom))
+  )
+  (hierarchical_label "Vout_HIGHPASS" (shape output) (at 108.585 83.82 180) (fields_autoplaced)
+    (effects (font (size 1.27 1.27)) (justify right))
+  )
+  (hierarchical_label "Vin_HIGHPASS" (shape input) (at 165.735 81.28 0) (fields_autoplaced)
+    (effects (font (size 1.27 1.27)) (justify left))
+  )
+  (symbol (lib_id "Device:R_US") (at 141.605 88.9 180) (unit 1)
+    (in_bom yes) (on_board yes) (dnp no) (fields_autoplaced)
+    (property "Reference" "R1" (at 143.51 88.265 0)
+      (effects (font (size 1.27 1.27)) (justify right))
+    )
+    (property "Value" "10K" (at 143.51 90.805 0)
+      (effects (font (size 1.27 1.27)) (justify right))
+    )
+    (property "Footprint" "" (at 140.589 88.646 90)
+      (effects (font (size 1.27 1.27)) hide)
+    )
+    (property "Datasheet" "~" (at 141.605 88.9 0)
+      (effects (font (size 1.27 1.27)) hide)
+    )
+    (pin "1")
+    (pin "2")
+    (instances
+      (project "Probe_PCB"
+        (path "/edde5bdb-d540-4f1f-a759-571037a8cf2c/7fb1114d-be17-466f-a435-ba2db15b5e3c"
+          (reference "R1") (unit 1)
+        )
+      )
+    )
+  )
+  (symbol (lib_id "Amplifier_Audio:OPA1622") (at 121.285 83.82 0) (mirror y) (unit 1)
+    (in_bom yes) (on_board yes) (dnp no)
+    (property "Reference" "U1" (at 121.285 70.485 0)
+      (effects (font (size 1.27 1.27)))
+    )
+    (property "Value" "OPA1622" (at 121.285 73.66 0)
+      (effects (font (size 1.27 1.27)))
+    )
+    (property "Footprint" "Package_SON:Texas_S-PVSON-N10" (at 121.285 93.98 0)
+      (effects (font (size 1.27 1.27)) hide)
+    )
+    (property "Datasheet" "http://www.ti.com/lit/ds/symlink/opa1622.pdf" (at 121.285 83.82 0)
+      (effects (font (size 1.27 1.27)) hide)
+    )
+    (pin "1")
+    (pin "10")
+    (pin "8")
+    (pin "9")
+    (pin "5")
+    (pin "6")
+    (pin "7")
+    (pin "11")
+    (pin "2")
+    (pin "3")
+    (pin "4")
+    (instances
+      (project "Probe_PCB"
+        (path "/edde5bdb-d540-4f1f-a759-571037a8cf2c/7fb1114d-be17-466f-a435-ba2db15b5e3c"
+          (reference "U1") (unit 1)
+        )
+      )
+    )
+  )
+  (symbol (lib_id "power:GNDREF") (at 141.605 102.87 0) (unit 1)
+    (in_bom yes) (on_board yes) (dnp no) (fields_autoplaced)
+    (property "Reference" "#PWR03" (at 141.605 109.22 0)
+      (effects (font (size 1.27 1.27)) hide)
+    )
+    (property "Value" "GNDREF" (at 141.605 107.95 0)
+      (effects (font (size 1.27 1.27)))
+    )
+    (property "Footprint" "" (at 141.605 102.87 0)
+      (effects (font (size 1.27 1.27)) hide)
+    )
+    (property "Datasheet" "" (at 141.605 102.87 0)
+      (effects (font (size 1.27 1.27)) hide)
+    )
+    (pin "1")
+    (instances
+      (project "Probe_PCB"
+        (path "/edde5bdb-d540-4f1f-a759-571037a8cf2c/7fb1114d-be17-466f-a435-ba2db15b5e3c"
+          (reference "#PWR03") (unit 1)
+        )
+      )
+    )
+  )
+  (symbol (lib_id "Device:C") (at 153.035 81.28 90) (unit 1)
+    (in_bom yes) (on_board yes) (dnp no) (fields_autoplaced)
+    (property "Reference" "C2" (at 153.035 74.93 90)
+      (effects (font (size 1.27 1.27)))
+    )
+    (property "Value" "100 uF" (at 153.035 77.47 90)
+      (effects (font (size 1.27 1.27)))
+    )
+    (property "Footprint" "" (at 156.845 80.3148 0)
+      (effects (font (size 1.27 1.27)) hide)
+    )
+    (property "Datasheet" "~" (at 153.035 81.28 0)
+      (effects (font (size 1.27 1.27)) hide)
+    )
+    (pin "1")
+    (pin "2")
+    (instances
+      (project "Probe_PCB"
+        (path "/edde5bdb-d540-4f1f-a759-571037a8cf2c/7fb1114d-be17-466f-a435-ba2db15b5e3c"
+          (reference "C2") (unit 1)
+        )
+      )
+    )
+  )
 )
