File: KiCAD_project_folder/Probe_PCB/low_pass_filter.kicad_sch (KiCad schematic)
At the start: 0 parts

Commit message: added schematic for filters and amplifier
Parts:
- added C2: 31,90 uF, symbol Device:C
- added R1: 50, symbol Device:R_US
- added U1: OPA1622, Package_SON:Texas_S-PVSON-N10, symbol Amplifier_Audio:OPA1622
Connections:
- new net: C2.1, R1.2, U1.1 (+)
- new net GNDREF: C2.2
- new net Vin_LOWPASS: R1.1
- new net Vout_LOWPASS: U1.10 (-), U1.9
Other:
- note added: "RC network, low-pass, R = 50R , C = 31 uF and fc = 100 Hz"
Changed lines of the file:
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@@
 (kicad_sch (version 20230121) (generator eeschema)
   (paper "A4")
+  (junction (at 152.4 108.585) (diameter 0) (color 0 0 0 0)
+  )
+  (junction (at 152.4 86.995) (diameter 0) (color 0 0 0 0)
+  )
+  (junction (at 124.46 89.535) (diameter 0) (color 0 0 0 0)
+  )
+  (wire (pts (xy 119.38 89.535) (xy 124.46 89.535))
+    (stroke (width 0) (type default))
+  )
+  (wire (pts (xy 152.4 98.425) (xy 152.4 108.585))
+    (stroke (width 0) (type default))
+  )
+  (wire (pts (xy 152.4 86.995) (xy 160.02 86.995))
+    (stroke (width 0) (type default))
+  )
+  (wire (pts (xy 152.4 108.585) (xy 176.53 108.585))
+    (stroke (width 0) (type default))
+  )
+  (wire (pts (xy 119.38 108.585) (xy 152.4 108.585))
+    (stroke (width 0) (type default))
+  )
+  (wire (pts (xy 139.7 86.995) (xy 152.4 86.995))
+    (stroke (width 0) (type default))
+  )
+  (wire (pts (xy 167.64 86.995) (xy 176.53 86.995))
+    (stroke (width 0) (type default))
+  )
+  (wire (pts (xy 124.46 98.425) (xy 124.46 89.535))
+    (stroke (width 0) (type default))
+  )
+  (wire (pts (xy 124.46 98.425) (xy 142.875 98.425))
+    (stroke (width 0) (type default))
+  )
+  (wire (pts (xy 142.875 92.075) (xy 142.875 98.425))
+    (stroke (width 0) (type default))
+  )
+  (wire (pts (xy 152.4 86.995) (xy 152.4 90.805))
+    (stroke (width 0) (type default))
+  )
+  (wire (pts (xy 142.875 92.075) (xy 139.7 92.075))
+    (stroke (width 0) (type default))
+  )
+  (rectangle (start 74.295 57.785) (end 219.075 137.795)
+    (stroke (width 0) (type default))
+    (fill (type none))
+  )
+  (text "RC network, low-pass, R = 50R , C = 31 uF and fc = 100 Hz"
+    (at 74.295 55.245 0)
+    (effects (font (size 1.27 1.27)) (justify left bottom))
+  )
+  (hierarchical_label "Vin_LOWPASS" (shape input) (at 176.53 86.995 0) (fields_autoplaced)
+    (effects (font (size 1.27 1.27)) (justify left))
+  )
+  (hierarchical_label "Vout_LOWPASS" (shape output) (at 119.38 89.535 180) (fields_autoplaced)
+    (effects (font (size 1.27 1.27)) (justify right))
+  )
+  (symbol (lib_id "Amplifier_Audio:OPA1622") (at 132.08 89.535 0) (mirror y) (unit 1)
+    (in_bom yes) (on_board yes) (dnp no)
+    (property "Reference" "U1" (at 132.08 76.2 0)
+      (effects (font (size 1.27 1.27)))
+    )
+    (property "Value" "OPA1622" (at 132.08 79.375 0)
+      (effects (font (size 1.27 1.27)))
+    )
+    (property "Footprint" "Package_SON:Texas_S-PVSON-N10" (at 132.08 99.695 0)
+      (effects (font (size 1.27 1.27)) hide)
+    )
+    (property "Datasheet" "http://www.ti.com/lit/ds/symlink/opa1622.pdf" (at 132.08 89.535 0)
+      (effects (font (size 1.27 1.27)) hide)
+    )
+    (pin "1")
+    (pin "10")
+    (pin "8")
+    (pin "9")
+    (pin "5")
+    (pin "6")
+    (pin "7")
+    (pin "11")
+    (pin "2")
+    (pin "3")
+    (pin "4")
+    (instances
+      (project "Probe_PCB"
+        (path "/edde5bdb-d540-4f1f-a759-571037a8cf2c/7fb1114d-be17-466f-a435-ba2db15b5e3c"
+          (reference "U1") (unit 1)
+        )
+        (path "/edde5bdb-d540-4f1f-a759-571037a8cf2c/5be9acd6-26f1-42dc-a981-07b70e893376"
+          (reference "U3") (unit 1)
+        )
+      )
+    )
+  )
+  (symbol (lib_id "Device:R_US") (at 163.83 86.995 270) (unit 1)
+    (in_bom yes) (on_board yes) (dnp no) (fields_autoplaced)
+    (property "Reference" "R1" (at 163.83 81.915 90)
+      (effects (font (size 1.27 1.27)))
+    )
+    (property "Value" "50" (at 163.83 84.455 90)
+      (effects (font (size 1.27 1.27)))
+    )
+    (property "Footprint" "" (at 163.576 88.011 90)
+      (effects (font (size 1.27 1.27)) hide)
+    )
+    (property "Datasheet" "~" (at 163.83 86.995 0)
+      (effects (font (size 1.27 1.27)) hide)
+    )
+    (pin "1")
+    (pin "2")
+    (instances
+      (project "Probe_PCB"
+        (path "/edde5bdb-d540-4f1f-a759-571037a8cf2c/7fb1114d-be17-466f-a435-ba2db15b5e3c"
+          (reference "R1") (unit 1)
+        )
+        (path "/edde5bdb-d540-4f1f-a759-571037a8cf2c/5be9acd6-26f1-42dc-a981-07b70e893376"
+          (reference "R6") (unit 1)
+        )
+      )
+    )
+  )
+  (symbol (lib_id "Device:C") (at 152.4 94.615 0) (unit 1)
+    (in_bom yes) (on_board yes) (dnp no) (fields_autoplaced)
+    (property "Reference" "C2" (at 156.21 93.98 0)
+      (effects (font (size 1.27 1.27)) (justify left))
+    )
+    (property "Value" "31,90 uF" (at 156.21 96.52 0)
+      (effects (font (size 1.27 1.27)) (justify left))
+    )
+    (property "Footprint" "" (at 153.3652 98.425 0)
+      (effects (font (size 1.27 1.27)) hide)
+    )
+    (property "Datasheet" "~" (at 152.4 94.615 0)
+      (effects (font (size 1.27 1.27)) hide)
+    )
+    (pin "1")
+    (pin "2")
+    (instances
+      (project "Probe_PCB"
+        (path "/edde5bdb-d540-4f1f-a759-571037a8cf2c/7fb1114d-be17-466f-a435-ba2db15b5e3c"
+          (reference "C2") (unit 1)
+        )
+        (path "/edde5bdb-d540-4f1f-a759-571037a8cf2c/5be9acd6-26f1-42dc-a981-07b70e893376"
+          (reference "C3") (unit 1)
+        )
+      )
+    )
+  )
+  (symbol (lib_id "power:GNDREF") (at 152.4 108.585 0) (unit 1)
+    (in_bom yes) (on_board yes) (dnp no) (fields_autoplaced)
+    (property "Reference" "#PWR03" (at 152.4 114.935 0)
+      (effects (font (size 1.27 1.27)) hide)
+    )
+    (property "Value" "GNDREF" (at 152.4 113.665 0)
+      (effects (font (size 1.27 1.27)))
+    )
+    (property "Footprint" "" (at 152.4 108.585 0)
+      (effects (font (size 1.27 1.27)) hide)
+    )
+    (property "Datasheet" "" (at 152.4 108.585 0)
+      (effects (font (size 1.27 1.27)) hide)
+    )
+    (pin "1")
+    (instances
+      (project "Probe_PCB"
+        (path "/edde5bdb-d540-4f1f-a759-571037a8cf2c/7fb1114d-be17-466f-a435-ba2db15b5e3c"
+          (reference "#PWR03") (unit 1)
+        )
+        (path "/edde5bdb-d540-4f1f-a759-571037a8cf2c/5be9acd6-26f1-42dc-a981-07b70e893376"
+          (reference "#PWR04") (unit 1)
+        )
+      )
+    )
+  )
 )
