File: KiCAD_project_folder/Probe_PCB/signal_amplifier.kicad_sch (KiCad schematic)
At the start: 0 parts

Commit message: added schematic for filters and amplifier
Parts:
- added C2: 3,1831uF, symbol Device:C
- added R1: 10000, symbol Device:R_US
- added R1: 100, symbol Device:R_US
- added R1: 50, symbol Device:R_US
- added U1: OPA1622, Package_SON:Texas_S-PVSON-N10, symbol Amplifier_Audio:OPA1622
Connections:
- new net: R1.1, R1.1, U1.10 (-)
- new net: C2.1, R1.2, U1.1 (+)
- new net GNDREF: C2.2, R1.2
- new net Vin_amp: R1.1
- new net Vout_amp: R1.2, U1.9
Other:
- note added: "RC network, low-pass, R = 50R , C = 3,1831 uF and fc = 1000 Hz"
